Commit message: Moved wheels up to move cameras closer to ground & moved cameras further appart

File: src/my_robot_description/urdf/cameraBL.xacro (robot description, xacro)
@@ -22,5 +22,5 @@
         <parent link="base_link" />
         <child link="camera_linkBL" />
-        <origin xyz="0 0.1 ${base_height / 2.0 - 0.305}" rpy="0 ${pi/2} 0" />
+        <origin xyz="0 0.2 ${base_height / 2.0 - 0.305}" rpy="0 ${pi/2} 0" />
     </joint>
     <link name="camera_link_opticalBL" />

File: src/my_robot_description/urdf/cameraBR.xacro (robot description, xacro)
@@ -22,5 +22,5 @@
         <parent link="base_link" />
         <child link="camera_linkBR" />
-        <origin xyz="0 -0.1 ${base_height / 2.0 - 0.305}" rpy="0 ${pi/2} 0" />
+        <origin xyz="0 -0.2 ${base_height / 2.0 - 0.305}" rpy="0 ${pi/2} 0" />
     </joint>
     <link name="camera_link_opticalBR" />

File: src/my_robot_description/urdf/mobile_base.xacro (robot description, xacro)
@@ -191,5 +191,5 @@
         <parent link="base_link"/>
         <child link="rear_left_wheel_link"/>
-        <origin xyz="${(-(base_length + 0.01) / 2.0) + 0.2} 0.32 -0.2" rpy="0 0 0"/>
+        <origin xyz="${(-(base_length + 0.01) / 2.0) + 0.2} 0.32 -0.15" rpy="0 0 0"/>
         <axis xyz="0 1 0"/>
     </joint>
@@ -197,5 +197,5 @@
         <parent link="base_link"/>
         <child link="rear_right_wheel_link"/>
-        <origin xyz="${(-(base_length + 0.01) / 2.0) + 0.2} -0.32 -0.2" rpy="0 0 0"/>
+        <origin xyz="${(-(base_length + 0.01) / 2.0) + 0.2} -0.32 -0.15" rpy="0 0 0"/>
         <axis xyz="0 1 0"/>
     </joint>
@@ -206,5 +206,5 @@
         <parent link="base_link"/>
         <child link="front_right_wheel_link"/>
-        <origin xyz="${((base_length + 0.01) / 2.0) - 0.2} -0.32 -0.2" rpy="0 0 0"/>
+        <origin xyz="${((base_length + 0.01) / 2.0) - 0.2} -0.32 -0.15" rpy="0 0 0"/>
         <axis xyz="0 1 0"/>
     </joint>
@@ -230,5 +230,5 @@
         <parent link="base_link"/>
         <child link="front_left_wheel_link"/>
-        <origin xyz="${((base_length + 0.01) / 2.0) - 0.2} 0.32 -0.2" rpy="0 0 0"/>
+        <origin xyz="${((base_length + 0.01) / 2.0) - 0.2} 0.32 -0.15" rpy="0 0 0"/>
         <axis xyz="0 1 0"/>
     </joint>
