Commit message: Fixed colour camera topic name

File: src/my_robot_description/urdf/camera_colour.xacro (robot description, xacro)
@@ -4,5 +4,5 @@
     <xacro:property name="camera_width" value="0.1" />
     <xacro:property name="camera_height" value="0.05" />
-    <link name="camera_colour_link">
+    <link name="colour_camera_link">
         <visual>
             <geometry>
@@ -19,18 +19,18 @@
                            o_xyz="0 0 0" o_rpy="0 0 0" />
     </link>
-    <joint name="base_camera_colour_joint" type="fixed">
+    <joint name="base_colour_camera_joint" type="fixed">
         <parent link="base_link" />
-        <child link="camera_colour_link" />
+        <child link="colour_camera_link" />
         <!-- Positioned on top of the camera, facing forward (rpy="0 0 0") -->
         <origin xyz="${(base_length + camera_length) / 2.0} 0 ${base_height / 2.0 - 0.02}" rpy="0 0 0" />
     </joint>
-    <link name="camera_colour_link_optical" />
-    <joint name="camera_colour_optical_joint" type="fixed">
+    <link name="colour_camera_link_optical" />
+    <joint name="colour_camera_optical_joint" type="fixed">
         <origin xyz="0 0 0" rpy="${-pi/2} 0 ${-pi/2}"/>
-        <parent link="camera_colour_link"/>
-        <child link="camera_colour_link_optical"/>
+        <parent link="colour_camera_link"/>
+        <child link="colour_camera_link_optical"/>
     </joint>
-    <gazebo reference="camera_colour_link">
-        <sensor name="camera_colour" type="camera">
+    <gazebo reference="colour_camera_link">
+        <sensor name="colour_camera" type="camera">
             <camera>
                 <horizontal_fov>1.3962634</horizontal_fov>
@@ -49,14 +49,14 @@
                     <stddev>0.007</stddev>
                 </noise>
-                <optical_frame_id>camera_colour_link_optical</optical_frame_id>
-                <camera_info_topic>camera_colour/camera_info</camera_info_topic>
+                <optical_frame_id>colour_camera_link_optical</optical_frame_id>
+                <camera_info_topic>colour_camera/camera_info</camera_info_topic>
             </camera>
             <always_on>1</always_on>
             <update_rate>3</update_rate>
             <visualize>true</visualize>
-            <topic>camera_colour/image_raw</topic>
+            <topic>colour_camera/image_raw</topic>
             <plugin
                 filename="gz-sim-camera-system"
-                name="camera_colour_plugin"/>
+                name="colour_camera_plugin"/>
         </sensor>
     </gazebo>

Commit message: creating camera

File: src/my_robot_description/urdf/camera_colour.xacro (robot description, xacro)
@@ -1,8 +1,8 @@
 <?xml version="1.0"?>
 <robot xmlns:xacro="http://www.ros.org/wiki/xacro">
-    <xacro:property name="camera_length" value="0.01" />
-    <xacro:property name="camera_width" value="0.1" />
+    <xacro:property name="camera_length" value="0.002" />
+    <xacro:property name="camera_width" value="0.035" />
     <xacro:property name="camera_height" value="0.05" />
-    <link name="colour_camera_link">
+    <link name="camera_link">
         <visual>
             <geometry>
@@ -19,18 +19,18 @@
                            o_xyz="0 0 0" o_rpy="0 0 0" />
     </link>
-    <joint name="base_colour_camera_joint" type="fixed">
-        <parent link="base_link" />
-        <child link="colour_camera_link" />
+    <joint name="base_camera_joint" type="fixed">
+        <parent link="servo_link" />
+        <child link="camera_link" />
         <!-- Positioned on top of the camera, facing forward (rpy="0 0 0") -->
-        <origin xyz="${(base_length + camera_length) / 2.0} 0 ${base_height / 2.0 - 0.02}" rpy="0 0 0" />
+        <origin xyz="0.085 0 0.0825" rpy="1.047 0 0" />
     </joint>
-    <link name="colour_camera_link_optical" />
-    <joint name="colour_camera_optical_joint" type="fixed">
+    <link name="camera_link_optical" />
+    <joint name="optical_joint" type="fixed">
         <origin xyz="0 0 0" rpy="${-pi/2} 0 ${-pi/2}"/>
-        <parent link="colour_camera_link"/>
-        <child link="colour_camera_link_optical"/>
+        <parent link="camera_link"/>
+        <child link="camera_link_optical"/>
     </joint>
-    <gazebo reference="colour_camera_link">
-        <sensor name="colour_camera" type="camera">
+    <gazebo reference="camera_link">
+        <sensor name="camera" type="camera">
             <camera>
                 <horizontal_fov>1.3962634</horizontal_fov>
@@ -49,14 +49,14 @@
                     <stddev>0.007</stddev>
                 </noise>
-                <optical_frame_id>colour_camera_link_optical</optical_frame_id>
-                <camera_info_topic>colour_camera/camera_info</camera_info_topic>
+                <optical_frame_id>camera_link_optical</optical_frame_id>
+                <camera_info_topic>camera/camera_info</camera_info_topic>
             </camera>
             <always_on>1</always_on>
             <update_rate>3</update_rate>
             <visualize>true</visualize>
-            <topic>colour_camera/image_raw</topic>
+            <topic>camera/image_raw</topic>
             <plugin
                 filename="gz-sim-camera-system"
-                name="colour_camera_plugin"/>
+                name="camera_plugin"/>
         </sensor>
     </gazebo>

File: src/my_robot_description/urdf/my_robot.urdf.xacro (robot description, xacro)
@@ -4,5 +4,4 @@
     <xacro:include filename="mobile_base.xacro" />
     <xacro:include filename="mobile_base_gazebo.xacro" />
-    <xacro:include filename="camera.xacro" />
     <xacro:include filename="cameraBM.xacro" />
     <xacro:include filename="cameraBL.xacro" />

Commit message: adjustments to camera

File: src/my_robot_description/urdf/camera_colour.xacro (robot description, xacro)
@@ -23,5 +23,5 @@
         <child link="camera_link" />
         <!-- Positioned on top of the camera, facing forward (rpy="0 0 0") -->
-        <origin xyz="0.085 0 0.0825" rpy="1.047 0 0" />
+        <origin xyz="-0.005 0 0.06" rpy="0 1.047 0" />
     </joint>
     <link name="camera_link_optical" />

Commit message: adjustments

File: src/my_robot_description/urdf/camera_colour.xacro (robot description, xacro)
@@ -23,5 +23,5 @@
         <child link="camera_link" />
         <!-- Positioned on top of the camera, facing forward (rpy="0 0 0") -->
-        <origin xyz="-0.005 0 0.06" rpy="0 1.047 0" />
+        <origin xyz="-0.005 0 0.06" rpy="0 2.094 0" />
     </joint>
     <link name="camera_link_optical" />

File: src/my_robot_description/urdf/mobile_base.xacro (robot description, xacro)
@@ -45,6 +45,5 @@
             <parent link="base_link"/>
             <child link="servo_link"/>
-            <origin xyz="0.09 0 0.0225" rpy="0 0 0"/>
-            <!-- z was 0.045 -->
+            <origin xyz="0.09 0 0.0375" rpy="0 0 0"/>
             <axis xyz="0 0 1"/>
         </joint>

Commit message: x

File: src/my_robot_description/urdf/camera_colour.xacro (robot description, xacro)
@@ -23,5 +23,5 @@
         <child link="camera_link" />
         <!-- Positioned on top of the camera, facing forward (rpy="0 0 0") -->
-        <origin xyz="-0.005 0 0.06" rpy="0 2.094 0" />
+        <origin xyz="-0.005 0 0.06" rpy="0 1.745 0" />
     </joint>
     <link name="camera_link_optical" />

File: src/my_robot_description/urdf/mobile_base.xacro (robot description, xacro)
@@ -45,5 +45,5 @@
             <parent link="base_link"/>
             <child link="servo_link"/>
-            <origin xyz="0.09 0 0.0375" rpy="0 0 0"/>
+            <origin xyz="0.09 0 0.03" rpy="0 0 0"/>
             <axis xyz="0 0 1"/>
         </joint>

Commit message: camera + servo finished

File: src/my_robot_description/urdf/camera_colour.xacro (robot description, xacro)
@@ -23,5 +23,5 @@
         <child link="camera_link" />
         <!-- Positioned on top of the camera, facing forward (rpy="0 0 0") -->
-        <origin xyz="-0.005 0 0.06" rpy="0 1.745 0" />
+        <origin xyz="-0.005 0 0.06" rpy="0 2.793 0" />
     </joint>
     <link name="camera_link_optical" />
