Commit message: robot tag

File: src/my_robot_description/urdf/mobile_base_gazebo.xacro (robot description, xacro)
@@ -1,4 +1,5 @@
 <?xml version="1.0"?>
-<xacro:macro name="gazebo_file" params="bot_name" xmlns:xacro="http://www.ros.org/wiki/xacro">
+<robot xmlns:xacro="http://www.ros.org/wiki/xacro">
+<xacro:macro name="gazebo_file" params="bot_name" >
     <!-- Friction for wheels -->
     <gazebo reference="${bot_name}_rear_left_wheel_link">
@@ -45,2 +46,3 @@
     </gazebo>
 </xacro:macro>
+</robot>

Commit message: x

File: src/my_robot_description/urdf/mobile_base_gazebo.xacro (robot description, xacro)
@@ -1,48 +1,48 @@
 <?xml version="1.0"?>
 <robot xmlns:xacro="http://www.ros.org/wiki/xacro">
-<xacro:macro name="gazebo_file" params="bot_name" >
-    <!-- Friction for wheels -->
-    <gazebo reference="${bot_name}_rear_left_wheel_link">
-        <mu1 value="1" />
-        <mu2 value="1" />
-    </gazebo>
-    <gazebo reference="${bot_name}_rear_right_wheel_link">
-        <mu1 value="1" />
-        <mu2 value="1" />
-    </gazebo>
-     <gazebo reference="${bot_name}_front_left_wheel_link">
-        <mu1 value="1" />
-        <mu2 value="1" />
-    </gazebo>
-    <gazebo reference="${bot_name}_front_right_wheel_link">
-        <mu1 value="1" />
-        <mu2 value="1" />
-    </gazebo>
-    <!-- Differential Drive Plugin -->
-    <gazebo>
-        <plugin
-            filename="gz-sim-diff-drive-system"
-            name="gz::sim::systems::DiffDrive">
-            <left_joint>rear_left_wheel_joint</left_joint>
-            <right_joint>rear_right_wheel_joint</right_joint>
-            <wheel_separation>0.124</wheel_separation>
-            <wheel_radius>0.032</wheel_radius>
-            <max_wheel_torque>100</max_wheel_torque>
-            <max_wheel_acceleration>2.0</max_wheel_acceleration>
-            <frame_id>odom</frame_id>
-            <child_frame_id>base_footprint</child_frame_id>
-        </plugin>
-    </gazebo>
-    <!-- Joint State Publisher -->
-    <gazebo>
-        <plugin
-            filename="gz-sim-joint-state-publisher-system"
-            name="gz::sim::systems::JointStatePublisher">
-            <joint_name>${bot_name}_rear_left_wheel_joint</joint_name>
-            <joint_name>${bot_name}_rear_right_wheel_joint</joint_name>
-            <joint_name>${bot_name}_front_left_wheel_link</joint_name>
-            <joint_name>${bot_name}_front_right_wheel_link</joint_name>
-        </plugin>
-    </gazebo>
-</xacro:macro>
+    <xacro:macro name="gazebo_file" params="bot_name" >
+        <!-- Friction for wheels -->
+        <gazebo reference="${bot_name}_rear_left_wheel_link">
+            <mu1 value="1" />
+            <mu2 value="1" />
+        </gazebo>
+        <gazebo reference="${bot_name}_rear_right_wheel_link">
+            <mu1 value="1" />
+            <mu2 value="1" />
+        </gazebo>
+        <gazebo reference="${bot_name}_front_left_wheel_link">
+            <mu1 value="1" />
+            <mu2 value="1" />
+        </gazebo>
+        <gazebo reference="${bot_name}_front_right_wheel_link">
+            <mu1 value="1" />
+            <mu2 value="1" />
+        </gazebo>
+        <!-- Differential Drive Plugin -->
+        <gazebo>
+            <plugin
+                filename="gz-sim-diff-drive-system"
+                name="gz::sim::systems::DiffDrive">
+                <left_joint>${bot_name}_rear_left_wheel_joint</left_joint>
+                <right_joint>${bot_name}_rear_right_wheel_joint</right_joint>
+                <wheel_separation>0.124</wheel_separation>
+                <wheel_radius>0.032</wheel_radius>
+                <max_wheel_torque>100</max_wheel_torque>
+                <max_wheel_acceleration>2.0</max_wheel_acceleration>
+                <frame_id>odom</frame_id>
+                <child_frame_id>${bot_name}_base_footprint</child_frame_id>
+            </plugin>
+        </gazebo>
+        <!-- Joint State Publisher -->
+        <gazebo>
+            <plugin
+                filename="gz-sim-joint-state-publisher-system"
+                name="gz::sim::systems::JointStatePublisher">
+                <joint_name>${bot_name}_rear_left_wheel_joint</joint_name>
+                <joint_name>${bot_name}_rear_right_wheel_joint</joint_name>
+                <joint_name>${bot_name}_front_left_wheel_joint</joint_name>
+                <joint_name>${bot_name}_front_right_wheel_joint</joint_name>
+            </plugin>
+        </gazebo>
+    </xacro:macro>
 </robot>

File: src/my_robot_description/urdf/ultrasonic.xacro (robot description, xacro)
@@ -32,5 +32,5 @@
     </joint>
     <gazebo reference="${bot_name}_lidar_link">
-        <sensor type="ray" name="lidar_sensor">
+        <sensor type="ray" name="${bot_name}_lidar_sensor">
             <update_rate>10.0</update_rate>
             <ray>
@@ -54,6 +54,6 @@
                 <remapping>~/out:=scan</remapping>
             </ros>
-            <output_type>${bot_name}_sensor_msgs/LaserScan</output_type>
-            <frame_name>lidar_link</frame_name>
+            <output_type>sensor_msgs/LaserScan</output_type>
+            <frame_name>${bot_name}_lidar_link</frame_name>
             </plugin>
         </sensor>
