Commit message: x

File: src/my_robot_description/urdf/common_properties.xacro (robot description, xacro)
@@ -11,6 +11,6 @@
         <color rgba="0.5 0 0 1.0"/>
     </material>
-    <!-- Additional colors for your robot model -->
-    <material name="body_blue">
+    <!-- Robot Base Colour (Blue, Green, Yellow) -->
+    <material name="generic">
         <color rgba="0.09 0.46 0.71 1.0"/>
     </material>

File: src/my_robot_description/urdf/my_robot.urdf.xacro (robot description, xacro)
@@ -8,5 +8,5 @@
     <xacro:include filename="camera.xacro" />
     <xacro:include filename="wheel.xacro"/>
-    <xacro:arg name="bot_name" default="twix"/>
+    <xacro:arg name="bot_name" default="generic"/>
     <xacro:bot bot_name="$(arg bot_name)"/>
 </robot>
