Commit message: x

File: src/my_robot_description/urdf/wheel.xacro (robot description, xacro)
@@ -22,5 +22,5 @@
             <parent link="${bot_name}_base_link"/>
             <child link="${bot_name}_${prefix}_wheel_link"/>
-            <origin xyz="${invert_x*0.04} ${invert_y*(base_width/2.0) - 0.016} -0.005" rpy="0 0 0"/>
+            <origin xyz="${invert_x*0.04} ${invert_y*((base_width/2.0) - 0.016)} -0.005" rpy="0 0 0"/>
             <axis xyz="0 1 0"/>
         </joint>

Commit message: x

File: src/my_robot_description/urdf/wheel.xacro (robot description, xacro)
@@ -22,5 +22,5 @@
             <parent link="${bot_name}_base_link"/>
             <child link="${bot_name}_${prefix}_wheel_link"/>
-            <origin xyz="${invert_x*0.04} ${invert_y*((base_width/2.0) - 0.016)} -0.005" rpy="0 0 0"/>
+            <origin xyz="${invert_x*0.04} ${(invert_y*base_width/2.0) + (invert_y*0.016)} -0.005" rpy="0 0 0"/>
             <axis xyz="0 1 0"/>
         </joint>
