Commit message: qed nibza mill vm

File: src/my_robot_description/urdf/camera.xacro (robot description, xacro)
@@ -22,5 +22,5 @@
         <parent link="base_link" />
         <child link="camera_link" />
-        <origin xyz="${(base_length + camera_length) / 2.0} 0 ${base_height / 2.0 - 0.1}" rpy="0 0.4 0" />
+        <origin xyz="${(base_length + camera_length) / 2.0} 0 ${base_height / 2.0 - 0.1}" rpy="0 0.5 0" />
     </joint>
     <link name="camera_link_optical" />

Commit message: push to work from laptop

File: src/my_robot_description/urdf/camera.xacro (robot description, xacro)
@@ -22,5 +22,5 @@
         <parent link="base_link" />
         <child link="camera_link" />
-        <origin xyz="${(base_length + camera_length) / 2.0} 0 ${base_height / 2.0 - 0.1}" rpy="0 0.5 0" />
+        <origin xyz="${(base_length + camera_length) / 2.0} 0 ${base_height / 2.0 - 0.1}" rpy="0 0.6 0" />
     </joint>
     <link name="camera_link_optical" />

Commit message: model adjustments

File: src/my_robot_description/urdf/camera.xacro (robot description, xacro)
@@ -2,6 +2,6 @@
 <robot xmlns:xacro="http://www.ros.org/wiki/xacro">
     <xacro:property name="camera_length" value="0.002" />
-    <xacro:property name="camera_width" value="0.035" />
-    <xacro:property name="camera_height" value="0.05" />
+    <xacro:property name="camera_width" value="0.031" />
+    <xacro:property name="camera_height" value="0.046" />
     <link name="camera_link">
         <visual>
@@ -22,6 +22,5 @@
         <parent link="servo_link" />
         <child link="camera_link" />
-        <!-- Positioned on top of the camera, facing forward (rpy="0 0 0") -->
-        <origin xyz="-0.005 0 0.06" rpy="0 2.793 0" />
+        <origin xyz="-0.016 0 0.082" rpy="0 2.793 3.142" />
     </joint>
     <link name="camera_link_optical" />

File: src/my_robot_description/urdf/ultrasonic.xacro (robot description, xacro)
@@ -1,5 +1,5 @@
 <?xml version="1.0"?>
 <robot xmlns:xacro="http://www.ros.org/wiki/xacro">
-    <xacro:property name="lidar_length" value="0.002" />
+    <xacro:property name="lidar_length" value="0.024" />
     <xacro:property name="lidar_width" value="0.05" />
     <xacro:property name="lidar_height" value="0.023" />
@@ -22,6 +22,5 @@
         <parent link="servo_link" />
         <child link="lidar_link" />
-        <!-- Positioned on top of the lidar, facing forward (rpy="0 0 0") -->
-        <origin xyz="-0.005 0 0.02" rpy="0 0 0" />
+        <origin xyz="-0.0025 0 0.026" rpy="0 0 0" />
     </joint>
     <link name="lidar_link_optical" />

Commit message: model finished

File: src/my_robot_description/urdf/camera.xacro (robot description, xacro)
@@ -22,5 +22,5 @@
         <parent link="servo_link" />
         <child link="camera_link" />
-        <origin xyz="-0.016 0 0.082" rpy="0 2.793 3.142" />
+        <origin xyz="-0.016 0 0.082" rpy="0 0.349 3.142" />
     </joint>
     <link name="camera_link_optical" />

Commit message: started duplication of xacro

File: src/my_robot_description/urdf/camera.xacro (robot description, xacro)
@@ -4,5 +4,5 @@
     <xacro:property name="camera_width" value="0.031" />
     <xacro:property name="camera_height" value="0.046" />
-    <link name="camera_link">
+    <link name="${bot_name}_camera_link">
         <visual>
             <geometry>
@@ -19,17 +19,17 @@
                            o_xyz="0 0 0" o_rpy="0 0 0" />
     </link>
-    <joint name="base_camera_joint" type="fixed">
-        <parent link="servo_link" />
-        <child link="camera_link" />
+    <joint name="${bot_name}_base_camera_joint" type="fixed">
+        <parent link="${bot_name}_servo_link" />
+        <child link="${bot_name}_camera_link" />
         <origin xyz="-0.016 0 0.082" rpy="0 0.349 3.142" />
     </joint>
-    <link name="camera_link_optical" />
-    <joint name="optical_joint" type="fixed">
+    <link name="${bot_name}_camera_link_optical" />
+    <joint name="${bot_name}_optical_joint" type="fixed">
         <origin xyz="0 0 0" rpy="${-pi/2} 0 ${-pi/2}"/>
-        <parent link="camera_link"/>
-        <child link="camera_link_optical"/>
+        <parent link="${bot_name}_camera_link"/>
+        <child link="${bot_name}_camera_link_optical"/>
     </joint>
-    <gazebo reference="camera_link">
-        <sensor name="camera" type="camera">
+    <gazebo reference="${bot_name}_camera_link">
+        <sensor name="${bot_name}_camera" type="camera">
             <camera>
                 <horizontal_fov>1.3962634</horizontal_fov>
@@ -49,10 +49,10 @@
                 </noise>
                 <optical_frame_id>camera_link_optical</optical_frame_id>
-                <camera_info_topic>camera/camera_info</camera_info_topic>
+                <camera_info_topic>${bot_name}_camera/camera_info</camera_info_topic>
             </camera>
             <always_on>1</always_on>
             <update_rate>3</update_rate>
             <visualize>true</visualize>
-            <topic>camera/image_raw</topic>
+            <topic>${bot_name}_camera/image_raw</topic>
             <plugin
                 filename="gz-sim-camera-system"

File: src/my_robot_description/urdf/common_properties.xacro (robot description, xacro)
@@ -14,4 +14,10 @@
     <material name="body_blue">
         <color rgba="0.09 0.46 0.71 1.0"/>
+    </material>
+    <material name="twix">
+        <color rgba="1 1 0 1.0"/>
+    </material>
+    <material name="twirl">
+        <color rgba="0 1 0 1.0"/>
     </material>
     <material name="accent_orange">

File: src/my_robot_description/urdf/ir.xacro (robot description, xacro)
@@ -4,5 +4,5 @@
     <xacro:property name="ir_width" value="0.045" />
     <xacro:property name="ir_height" value="0.03" />
-    <link name="ir_link">
+    <link name="${bot_name}_ir_link">
         <visual>
             <geometry>
@@ -19,17 +19,17 @@
                            o_xyz="0 0 0" o_rpy="0 0 0" />
     </link>
-    <joint name="base_ir_joint" type="fixed">
-        <parent link="base_link" />
-        <child link="ir_link" />
+    <joint name="${bot_name}_base_ir_joint" type="fixed">
+        <parent link="${bot_name}_base_link" />
+        <child link="${bot_name}_ir_link" />
         <origin xyz="0.084 0 -0.0275" rpy="0 ${pi/2} 0" />
     </joint>
-    <link name="ir_link_optical" />
-    <joint name="ir_optical_joint" type="fixed">
+    <link name="${bot_name}_ir_link_optical" />
+    <joint name="${bot_name}_ir_optical_joint" type="fixed">
         <origin xyz="0 0 0" rpy="${-pi/2} 0 ${-pi/2}"/>
-        <parent link="ir_link"/>
-        <child link="ir_link_optical"/>
+        <parent link="${bot_name}_ir_link"/>
+        <child link="${bot_name}_ir_link_optical"/>
     </joint>
-    <gazebo reference="ir_link">
-        <sensor name="ir" type="camera">
+    <gazebo reference="${bot_name}_ir_link">
+        <sensor name="${bot_name}_ir" type="camera">
             <camera>
                 <horizontal_fov>1.3962634</horizontal_fov>
@@ -49,10 +49,10 @@
                 </noise>
                 <optical_frame_id>ir_link_optical</optical_frame_id>
-                <ir_info_topic>ir/camera_info</ir_info_topic>
+                <camera_info_topic>${bot_name}_ir/camera_info</camera_info_topic>
             </camera>
             <always_on>1</always_on>
             <update_rate>3</update_rate>
             <visualize>true</visualize>
-            <topic>ir/image_raw</topic>
+            <topic>${bot_name}_ir/image_raw</topic>
             <plugin
                 filename="gz-sim-camera-system"

File: src/my_robot_description/urdf/mobile_base.xacro (robot description, xacro)
@@ -1,5 +1,5 @@
 <?xml version="1.0"?>
-<!-- <xacro:macro name="bot" params="bot_name"> -->
-<robot xmlns:xacro="http://www.ros.org/wiki/xacro">
+<xacro:macro name="bot" params="bot_name">
+    <robot xmlns:xacro="http://www.ros.org/wiki/xacro">
         <!-- Updated properties to match your robot model -->
         <xacro:property name="base_length" value="0.21"/>
@@ -11,10 +11,9 @@
         <!-- Base Footprint (empty)   -->
         <!-- ========================= -->
-        <!-- <link name="${bot_name}_base_footprint"/> -->
-        <link name="base_footprint"/>
+        <link name="${bot_name}_base_footprint"/>
         <!-- Fixed transform to base_link (body_link in your model) -->
-        <joint name="base_joint" type="fixed">
-            <parent link="base_footprint"/>
-            <child link="base_link"/>
+        <joint name="${bot_name}_base_joint" type="fixed">
+            <parent link="${bot_name}_base_footprint"/>
+            <child link="${bot_name}_base_link"/>
             <origin xyz="0 0 0.02"/>
         </joint>
@@ -22,5 +21,5 @@
         <!-- Base link body  -->
         <!-- =============== -->
-        <link name="base_link">
+        <link name="${bot_name}_base_link">
             <visual>
                 <geometry>
@@ -28,7 +27,5 @@
                 </geometry>
                 <origin xyz="0 0 0"/>
-                <material name="body_blue">
-                    <color rgba="0.09 0.46 0.71 1.0"/>
-                </material>
+                <material name="${bot_name}"/>
             </visual>
             <collision>
@@ -42,11 +39,11 @@
         </link>
         <!-- servo -->
-        <joint name="servo_joint" type="continuous">
-            <parent link="base_link"/>
-            <child link="servo_link"/>
+        <joint name="${bot_name}_servo_joint" type="continuous">
+            <parent link="${bot_name}_base_link"/>
+            <child link="${bot_name}_servo_link"/>
             <origin xyz="0.076 0 0.03" rpy="0 0 0"/>
             <axis xyz="0 0 1"/>
         </joint>
-        <link name="servo_link">
+        <link name="${bot_name}_servo_link">
             <visual>
                 <origin xyz="0 0 0" rpy="0 0 0"/>
@@ -54,7 +51,5 @@
                     <box size="0.032 0.01 0.015"/>
                 </geometry>
-                <material name="accent_orange">
-                    <color rgba="0.95 0.47 0.14 1.0"/>
-                </material>
+                <material name="accent_orange"/>
             </visual>
             <collision>
@@ -70,6 +65,6 @@
         <!-- Rear Wheels (Driven)        -->
         <!-- ============================ -->
-        <xacro:macro name="wheel_link" params="prefix">
-            <link name="${prefix}_wheel_link">
+        <xacro:macro name="${bot_name}_wheel_link" params="prefix">
+            <link name="${bot_name}_${prefix}_wheel_link">
                 <visual>
                     <geometry>
@@ -77,7 +72,5 @@
                     </geometry>
                     <origin xyz="0 0 0" rpy="${pi/2} 0 0"/>
-                    <material name="rubber_black">
-                        <color rgba="0.06 0.06 0.06 1.0"/>
-                    </material>
+                    <material name="rubber_black"/>
                 </visual>
                 <collision>
@@ -95,30 +88,28 @@
         <xacro:wheel_link prefix="front_left"/>
         <xacro:wheel_link prefix="front_right"/>
-        <joint name="rear_left_wheel_joint" type="continuous">
-            <parent link="base_link"/>
-            <child link="rear_left_wheel_link"/>
+        <joint name="${bot_name}_rear_left_wheel_joint" type="continuous">
+            <parent link="${bot_name}_base_link"/>
+            <child link="${bot_name}_rear_left_wheel_link"/>
             <origin xyz="-0.04 ${-(base_width/2.0) - 0.016} -0.005" rpy="0 0 0"/>
             <axis xyz="0 1 0"/>
         </joint>
-        <joint name="rear_right_wheel_joint" type="continuous">
-            <parent link="base_link"/>
-            <child link="rear_right_wheel_link"/>
+        <joint name="${bot_name}_rear_right_wheel_joint" type="continuous">
+            <parent link="${bot_name}_base_link"/>
+            <child link="${bot_name}_rear_right_wheel_link"/>
             <origin xyz="-0.04 ${(base_width/2.0) + 0.016} -0.005" rpy="0 0 0"/>
             <axis xyz="0 1 0"/>
         </joint>
-        <joint name="front_left_wheel_joint" type="continuous">
-            <parent link="base_link"/>
-            <child link="front_left_wheel_link"/>
+        <joint name="${bot_name}_front_left_wheel_joint" type="continuous">
+            <parent link="${bot_name}_base_link"/>
+            <child link="${bot_name}_front_left_wheel_link"/>
             <origin xyz="0.04 ${-(base_width/2.0) - 0.016} -0.005" rpy="0 0 0"/>
             <axis xyz="0 1 0"/>
         </joint>
-        <joint name="front_right_wheel_joint" type="continuous">
-            <parent link="base_link"/>
-            <child link="front_right_wheel_link"/>
+        <joint name="${bot_name}_front_right_wheel_joint" type="continuous">
+            <parent link="${bot_name}_base_link"/>
+            <child link="${bot_name}_front_right_wheel_link"/>
             <origin xyz="0.04 ${(base_width/2.0) + 0.016} -0.005" rpy="0 0 0"/>
             <axis xyz="0 1 0"/>
         </joint>
-</robot>
-<!-- </xacro:macro> -->
-<!-- <xacro:rear_wheel_link bot_name="twix"/>
-<xacro:rear_wheel_link bot_name="twirl"/> -->
+    </robot>
+</xacro:macro>

File: src/my_robot_description/urdf/my_robot.urdf.xacro (robot description, xacro)
@@ -8,2 +8,4 @@
     <xacro:include filename="camera.xacro" />
 </robot>
+<xacro:bot bot_name="twix"/>
+<xacro:bot bot_name="twirl"/>

File: src/my_robot_description/urdf/ultrasonic.xacro (robot description, xacro)
@@ -4,5 +4,5 @@
     <xacro:property name="lidar_width" value="0.05" />
     <xacro:property name="lidar_height" value="0.023" />
-    <link name="lidar_link">
+    <link name="${bot_name}_lidar_link">
         <visual>
             <geometry>
@@ -19,16 +19,16 @@
                            o_xyz="0 0 0" o_rpy="0 0 0" />
     </link>
-    <joint name="base_lidar_joint" type="fixed">
-        <parent link="servo_link" />
-        <child link="lidar_link" />
+    <joint name="${bot_name}_base_lidar_joint" type="fixed">
+        <parent link="${bot_name}_servo_link" />
+        <child link="${bot_name}_lidar_link" />
         <origin xyz="-0.0025 0 0.026" rpy="0 0 0" />
     </joint>
-    <link name="lidar_link_optical" />
-    <joint name="lidar_optical_joint" type="fixed">
+    <link name="${bot_name}_lidar_link_optical" />
+    <joint name="${bot_name}_lidar_optical_joint" type="fixed">
         <origin xyz="0 0 0" rpy="${-pi/2} 0 ${-pi/2}"/>
-        <parent link="lidar_link"/>
-        <child link="lidar_link_optical"/>
+        <parent link="${bot_name}_lidar_link"/>
+        <child link="${bot_name}_lidar_link_optical"/>
     </joint>
-    <gazebo reference="lidar_link">
+    <gazebo reference="${bot_name}_lidar_link">
         <sensor type="ray" name="lidar_sensor">
             <update_rate>10.0</update_rate>
@@ -53,5 +53,5 @@
                 <remapping>~/out:=scan</remapping>
             </ros>
-            <output_type>sensor_msgs/LaserScan</output_type>
+            <output_type>${bot_name}_sensor_msgs/LaserScan</output_type>
             <frame_name>lidar_link</frame_name>
             </plugin>

Commit message: adjustments to duplication

File: src/my_robot_description/urdf/camera.xacro (robot description, xacro)
@@ -1,4 +1,4 @@
 <?xml version="1.0"?>
-<robot xmlns:xacro="http://www.ros.org/wiki/xacro">
+<xacro:macro name="camera_sensor" params="bot_name">
     <xacro:property name="camera_length" value="0.002" />
     <xacro:property name="camera_width" value="0.031" />
@@ -48,5 +48,5 @@
                     <stddev>0.007</stddev>
                 </noise>
-                <optical_frame_id>camera_link_optical</optical_frame_id>
+                <optical_frame_id>${bot_name}_camera_link_optical</optical_frame_id>
                 <camera_info_topic>${bot_name}_camera/camera_info</camera_info_topic>
             </camera>
@@ -60,3 +60,3 @@
         </sensor>
     </gazebo>
-</robot>
+</xacro:macro>

File: src/my_robot_description/urdf/ir.xacro (robot description, xacro)
@@ -1,4 +1,4 @@
 <?xml version="1.0"?>
-<robot xmlns:xacro="http://www.ros.org/wiki/xacro">
+<xacro:macro name="ir_sensor" params="bot_name">
     <xacro:property name="ir_length" value="0.01" />
     <xacro:property name="ir_width" value="0.045" />
@@ -48,5 +48,5 @@
                     <stddev>0.007</stddev>
                 </noise>
-                <optical_frame_id>ir_link_optical</optical_frame_id>
+                <optical_frame_id>${bot_name}_ir_link_optical</optical_frame_id>
                 <camera_info_topic>${bot_name}_ir/camera_info</camera_info_topic>
             </camera>
@@ -57,6 +57,6 @@
             <plugin
                 filename="gz-sim-camera-system"
-                name="camera_plugin"/>
+                name="gz::sim::systems::Camera"/>
         </sensor>
     </gazebo>
-</robot>
+</xacro:macro>

File: src/my_robot_description/urdf/mobile_base.xacro (robot description, xacro)
@@ -1,5 +1,4 @@
 <?xml version="1.0"?>
 <xacro:macro name="bot" params="bot_name">
-    <robot xmlns:xacro="http://www.ros.org/wiki/xacro">
         <!-- Updated properties to match your robot model -->
         <xacro:property name="base_length" value="0.21"/>
@@ -112,4 +111,6 @@
             <axis xyz="0 1 0"/>
         </joint>
-    </robot>
+    <xacro:ir_sensor botname="${bot_name}"/>
+    <xacro:camera_sensor botname="${bot_name}"/>
+    <xacro:ultrasonic_sensor botname="${bot_name}"/>
 </xacro:macro>

File: src/my_robot_description/urdf/my_robot.urdf.xacro (robot description, xacro)
@@ -7,5 +7,5 @@
     <xacro:include filename="ultrasonic.xacro" />
     <xacro:include filename="camera.xacro" />
+    <xacro:bot bot_name="twix"/>
+    <xacro:bot bot_name="twirl"/>
 </robot>
-<xacro:bot bot_name="twix"/>
-<xacro:bot bot_name="twirl"/>

File: src/my_robot_description/urdf/ultrasonic.xacro (robot description, xacro)
@@ -1,4 +1,4 @@
 <?xml version="1.0"?>
-<robot xmlns:xacro="http://www.ros.org/wiki/xacro">
+<xacro:macro name="ultrasonic_sensor" params="bot_name">
     <xacro:property name="lidar_length" value="0.024" />
     <xacro:property name="lidar_width" value="0.05" />
@@ -58,3 +58,3 @@
         </sensor>
     </gazebo>
-</robot>
+</xacro:macro>

Commit message: changes

File: src/my_robot_description/urdf/camera.xacro (robot description, xacro)
@@ -1,4 +1,4 @@
 <?xml version="1.0"?>
-<xacro:macro name="camera_sensor" params="bot_name">
+<xacro:macro name="camera_sensor" params="bot_name" xmlns:xacro="http://www.ros.org/wiki/xacro">
     <xacro:property name="camera_length" value="0.002" />
     <xacro:property name="camera_width" value="0.031" />

File: src/my_robot_description/urdf/ir.xacro (robot description, xacro)
@@ -1,4 +1,4 @@
 <?xml version="1.0"?>
-<xacro:macro name="ir_sensor" params="bot_name">
+<xacro:macro name="ir_sensor" params="bot_name" xmlns:xacro="http://www.ros.org/wiki/xacro">
     <xacro:property name="ir_length" value="0.01" />
     <xacro:property name="ir_width" value="0.045" />

File: src/my_robot_description/urdf/mobile_base.xacro (robot description, xacro)
@@ -1,4 +1,4 @@
 <?xml version="1.0"?>
-<xacro:macro name="bot" params="bot_name">
+<xacro:macro name="bot" params="bot_name" xmlns:xacro="http://www.ros.org/wiki/xacro">
         <!-- Updated properties to match your robot model -->
         <xacro:property name="base_length" value="0.21"/>
@@ -111,6 +111,7 @@
             <axis xyz="0 1 0"/>
         </joint>
-    <xacro:ir_sensor botname="${bot_name}"/>
-    <xacro:camera_sensor botname="${bot_name}"/>
-    <xacro:ultrasonic_sensor botname="${bot_name}"/>
+    <xacro:ir_sensor bot_name="${bot_name}"/>
+    <xacro:camera_sensor bot_name="${bot_name}"/>
+    <xacro:ultrasonic_sensor bot_name="${bot_name}"/>
+    <xacro:gazebo_file bot_name="${bot_name}"/>
 </xacro:macro>

File: src/my_robot_description/urdf/mobile_base_gazebo.xacro (robot description, xacro)
@@ -1,18 +1,18 @@
 <?xml version="1.0"?>
-<robot xmlns:xacro="http://www.ros.org/wiki/xacro">
+<xacro:macro name="gazebo_file" params="bot_name" xmlns:xacro="http://www.ros.org/wiki/xacro">
     <!-- Friction for wheels -->
-    <gazebo reference="rear_left_wheel_link">
+    <gazebo reference="${bot_name}_rear_left_wheel_link">
         <mu1 value="1" />
         <mu2 value="1" />
     </gazebo>
-    <gazebo reference="rear_right_wheel_link">
+    <gazebo reference="${bot_name}_rear_right_wheel_link">
         <mu1 value="1" />
         <mu2 value="1" />
     </gazebo>
-     <gazebo reference="front_left_wheel_link">
+     <gazebo reference="${bot_name}_front_left_wheel_link">
         <mu1 value="1" />
         <mu2 value="1" />
     </gazebo>
-    <gazebo reference="right_right_wheel_link">
+    <gazebo reference="${bot_name}_front_right_wheel_link">
         <mu1 value="1" />
         <mu2 value="1" />
@@ -38,9 +38,9 @@
             filename="gz-sim-joint-state-publisher-system"
             name="gz::sim::systems::JointStatePublisher">
-            <joint_name>rear_left_wheel_joint</joint_name>
-            <joint_name>rear_right_wheel_joint</joint_name>
-            <joint_name>front_left_wheel_link</joint_name>
-            <joint_name>front_right_wheel_link</joint_name>
+            <joint_name>${bot_name}_rear_left_wheel_joint</joint_name>
+            <joint_name>${bot_name}_rear_right_wheel_joint</joint_name>
+            <joint_name>${bot_name}_front_left_wheel_link</joint_name>
+            <joint_name>${bot_name}_front_right_wheel_link</joint_name>
         </plugin>
     </gazebo>
-</robot>
+</xacro:macro>

File: src/my_robot_description/urdf/ultrasonic.xacro (robot description, xacro)
@@ -1,4 +1,4 @@
 <?xml version="1.0"?>
-<xacro:macro name="ultrasonic_sensor" params="bot_name">
+<xacro:macro name="ultrasonic_sensor" params="bot_name" xmlns:xacro="http://www.ros.org/wiki/xacro">
     <xacro:property name="lidar_length" value="0.024" />
     <xacro:property name="lidar_width" value="0.05" />
