Commit message: x

File: src/my_robot_description/urdf/camera.xacro (robot description, xacro)
@@ -1,4 +1,5 @@
 <?xml version="1.0"?>
-<xacro:macro name="camera_sensor" params="bot_name" xmlns:xacro="http://www.ros.org/wiki/xacro">
+<robot xmlns:xacro="http://www.ros.org/wiki/xacro">
+<xacro:macro name="camera_sensor" params="bot_name" >
     <xacro:property name="camera_length" value="0.002" />
     <xacro:property name="camera_width" value="0.031" />
@@ -61,2 +62,3 @@
     </gazebo>
 </xacro:macro>
+</robot>

File: src/my_robot_description/urdf/ir.xacro (robot description, xacro)
@@ -1,4 +1,5 @@
 <?xml version="1.0"?>
-<xacro:macro name="ir_sensor" params="bot_name" xmlns:xacro="http://www.ros.org/wiki/xacro">
+<robot xmlns:xacro="http://www.ros.org/wiki/xacro">
+<xacro:macro name="ir_sensor" params="bot_name" >
     <xacro:property name="ir_length" value="0.01" />
     <xacro:property name="ir_width" value="0.045" />
@@ -61,2 +62,3 @@
     </gazebo>
 </xacro:macro>
+</robot>

File: src/my_robot_description/urdf/mobile_base.xacro (robot description, xacro)
@@ -1,4 +1,5 @@
 <?xml version="1.0"?>
-<xacro:macro name="bot" params="bot_name" xmlns:xacro="http://www.ros.org/wiki/xacro">
+<robot xmlns:xacro="http://www.ros.org/wiki/xacro">
+<xacro:macro name="bot" params="bot_name" >
         <!-- Updated properties to match your robot model -->
         <xacro:property name="base_length" value="0.21"/>
@@ -116,2 +117,3 @@
     <xacro:gazebo_file bot_name="${bot_name}"/>
 </xacro:macro>
+</robot>

File: src/my_robot_description/urdf/ultrasonic.xacro (robot description, xacro)
@@ -1,4 +1,5 @@
 <?xml version="1.0"?>
-<xacro:macro name="ultrasonic_sensor" params="bot_name" xmlns:xacro="http://www.ros.org/wiki/xacro">
+<robot xmlns:xacro="http://www.ros.org/wiki/xacro">
+<xacro:macro name="ultrasonic_sensor" params="bot_name">
     <xacro:property name="lidar_length" value="0.024" />
     <xacro:property name="lidar_width" value="0.05" />
@@ -59,2 +60,3 @@
     </gazebo>
 </xacro:macro>
+</robot>

Commit message: fixing camera and ir

File: src/my_robot_description/urdf/camera.xacro (robot description, xacro)
@@ -27,5 +27,5 @@
     <link name="${bot_name}_camera_link_optical" />
     <joint name="${bot_name}_optical_joint" type="fixed">
-        <origin xyz="0 0 0" rpy="${-pi/2} 0 ${-pi/2}"/>
+        <origin xyz="0 0 0" rpy="0 0 {pi}"/>
         <parent link="${bot_name}_camera_link"/>
         <child link="${bot_name}_camera_link_optical"/>
@@ -41,5 +41,5 @@
                 </image>
                 <clip>
-                    <near>0.1</near>
+                    <near>0.0001</near>
                     <far>15</far>
                 </clip>

File: src/my_robot_description/urdf/ir.xacro (robot description, xacro)
@@ -41,5 +41,5 @@
                 </image>
                 <clip>
-                    <near>0.1</near>
+                    <near>0.001</near>
                     <far>15</far>
                 </clip>

Commit message: x

File: src/my_robot_description/urdf/camera.xacro (robot description, xacro)
@@ -27,5 +27,5 @@
     <link name="${bot_name}_camera_link_optical" />
     <joint name="${bot_name}_optical_joint" type="fixed">
-        <origin xyz="0 0 0" rpy="0 0 {pi}"/>
+        <origin xyz="0 0 0" rpy="0 0 ${pi}"/>
         <parent link="${bot_name}_camera_link"/>
         <child link="${bot_name}_camera_link_optical"/>

Commit message: camera sensors fixed

File: src/my_robot_description/urdf/camera.xacro (robot description, xacro)
@@ -23,9 +23,9 @@
         <parent link="${bot_name}_servo_link" />
         <child link="${bot_name}_camera_link" />
-        <origin xyz="-0.016 0 0.082" rpy="0 0.349 3.142" />
+        <origin xyz="-0.016 0 0.082" rpy="0 0.349 0" />
     </joint>
     <link name="${bot_name}_camera_link_optical" />
     <joint name="${bot_name}_optical_joint" type="fixed">
-        <origin xyz="0 0 0" rpy="0 0 ${pi}"/>
+        <origin xyz="0 0 0" rpy="0 0 0"/>
         <parent link="${bot_name}_camera_link"/>
         <child link="${bot_name}_camera_link_optical"/>

Commit message: x3 cameras on each robot for IR sensor

File: src/my_robot_description/urdf/camera.xacro (robot description, xacro)
@@ -1,64 +1,71 @@
 <?xml version="1.0"?>
 <robot xmlns:xacro="http://www.ros.org/wiki/xacro">
-<xacro:macro name="camera_sensor" params="bot_name" >
-    <xacro:property name="camera_length" value="0.002" />
-    <xacro:property name="camera_width" value="0.031" />
-    <xacro:property name="camera_height" value="0.046" />
-    <link name="${bot_name}_camera_link">
-        <visual>
-            <geometry>
-                <box size="${camera_length} ${camera_width} ${camera_height}" />
-            </geometry>
-            <material name="grey" />
-        </visual>
-        <collision>
-            <geometry>
-                <box size="${camera_length} ${camera_width} ${camera_height}" />
-            </geometry>
-        </collision>
-        <xacro:box_inertia m="0.1" x="${camera_length}" y="${camera_width}" z="${camera_height}"
-                           o_xyz="0 0 0" o_rpy="0 0 0" />
-    </link>
-    <joint name="${bot_name}_base_camera_joint" type="fixed">
-        <parent link="${bot_name}_servo_link" />
-        <child link="${bot_name}_camera_link" />
-        <origin xyz="-0.016 0 0.082" rpy="0 0.349 0" />
-    </joint>
-    <link name="${bot_name}_camera_link_optical" />
-    <joint name="${bot_name}_optical_joint" type="fixed">
-        <origin xyz="0 0 0" rpy="0 0 0"/>
-        <parent link="${bot_name}_camera_link"/>
-        <child link="${bot_name}_camera_link_optical"/>
-    </joint>
-    <gazebo reference="${bot_name}_camera_link">
-        <sensor name="${bot_name}_camera" type="camera">
-            <camera>
-                <horizontal_fov>1.3962634</horizontal_fov>
-                <image>
-                    <width>640</width>
-                    <height>480</height>
-                    <format>R8G8B8</format>
-                </image>
-                <clip>
-                    <near>0.0001</near>
-                    <far>15</far>
-                </clip>
-                <noise>
-                    <type>gaussian</type>
-                    <mean>0.0</mean>
-                    <stddev>0.007</stddev>
-                </noise>
-                <optical_frame_id>${bot_name}_camera_link_optical</optical_frame_id>
-                <camera_info_topic>${bot_name}_camera/camera_info</camera_info_topic>
-            </camera>
-            <always_on>1</always_on>
-            <update_rate>3</update_rate>
-            <visualize>true</visualize>
-            <topic>${bot_name}_camera/image_raw</topic>
-            <plugin
-                filename="gz-sim-camera-system"
-                name="camera_plugin"/>
-        </sensor>
-    </gazebo>
-</xacro:macro>
+    <xacro:macro name="camera_sensor" params="bot_name position_name" >
+        <xacro:property name="camera_length" value="0.002" />
+        <xacro:property name="camera_width" value="0.031" />
+        <xacro:property name="camera_height" value="0.046" />
+        <xacro:property name="y_offset" value="0.0" />
+        <xacro:if value="${position_name == 'L'}">
+            <xacro:property name="y_offset" value="${camera_width}" />
+        </xacro:if>
+        <xacro:if value="${position_name == 'R'}">
+            <xacro:property name="y_offset" value="${-camera_width}" />
+        </xacro:if>
+        <link name="${bot_name}_camera_${position_name}_link">
+            <visual>
+                <geometry>
+                    <box size="${camera_length} ${camera_width} ${camera_height}" />
+                </geometry>
+                <material name="grey" />
+            </visual>
+            <collision>
+                <geometry>
+                    <box size="${camera_length} ${camera_width} ${camera_height}" />
+                </geometry>
+            </collision>
+            <xacro:box_inertia m="0.1" x="${camera_length}" y="${camera_width}" z="${camera_height}"
+                            o_xyz="0 0 0" o_rpy="0 0 0" />
+        </link>
+        <joint name="${bot_name}_${position_name}_base_camera_joint" type="fixed">
+            <parent link="${bot_name}_servo_link" />
+            <child link="${bot_name}_camera_${position_name}_link" />
+            <origin xyz="-0.016 ${y_offset} 0.082" rpy="0 0.349 0" />
+        </joint>
+        <link name="${bot_name}_camera_${position_name}_link_optical" />
+        <joint name="${bot_name}_${position_name}_optical_joint" type="fixed">
+            <origin xyz="0 0 0" rpy="0 0 0"/>
+            <parent link="${bot_name}_camera_${position_name}_link"/>
+            <child link="${bot_name}_camera_${position_name}_link_optical"/>
+        </joint>
+        <gazebo reference="${bot_name}_camera_${position_name}_link">
+            <sensor name="${bot_name}_camera_${position_name}" type="camera">
+                <camera>
+                    <horizontal_fov>1.3962634</horizontal_fov>
+                    <image>
+                        <width>640</width>
+                        <height>480</height>
+                        <format>R8G8B8</format>
+                    </image>
+                    <clip>
+                        <near>0.0001</near>
+                        <far>15</far>
+                    </clip>
+                    <noise>
+                        <type>gaussian</type>
+                        <mean>0.0</mean>
+                        <stddev>0.007</stddev>
+                    </noise>
+                    <optical_frame_id>${bot_name}_camera_${position_name}_link_optical</optical_frame_id>
+                    <camera_info_topic>${bot_name}_camera_${position_name}/camera_info</camera_info_topic>
+                </camera>
+                <always_on>1</always_on>
+                <update_rate>3</update_rate>
+                <visualize>true</visualize>
+                <topic>${bot_name}_camera_${position_name}/image_raw</topic>
+                <plugin
+                    filename="gz-sim-camera-system"
+                    name="camera_plugin"/>
+            </sensor>
+        </gazebo>
+    </xacro:macro>
 </robot>

File: src/my_robot_description/urdf/mobile_base.xacro (robot description, xacro)
@@ -69,5 +69,7 @@
         <!-- sensors -->
         <xacro:ir_sensor bot_name="${bot_name}"/>
-        <xacro:camera_sensor bot_name="${bot_name}"/>
+        <xacro:camera_sensor bot_name="${bot_name}" position_name="L" />
+        <xacro:camera_sensor bot_name="${bot_name}" position_name="M" />
+        <xacro:camera_sensor bot_name="${bot_name}" position_name="R" />
         <xacro:ultrasonic_sensor bot_name="${bot_name}"/>
         <xacro:mpu_sensor bot_name="${bot_name}"/>

Commit message: *

File: src/my_robot_description/urdf/camera.xacro (robot description, xacro)
@@ -1,16 +1,9 @@
 <?xml version="1.0"?>
 <robot xmlns:xacro="http://www.ros.org/wiki/xacro">
-    <xacro:macro name="camera_sensor" params="bot_name position_name" >
+    <xacro:macro name="camera_sensor" params="bot_name" >
         <xacro:property name="camera_length" value="0.002" />
         <xacro:property name="camera_width" value="0.031" />
         <xacro:property name="camera_height" value="0.046" />
-        <xacro:property name="y_offset" value="0.0" />
-        <xacro:if value="${position_name == 'L'}">
-            <xacro:property name="y_offset" value="${camera_width}" />
-        </xacro:if>
-        <xacro:if value="${position_name == 'R'}">
-            <xacro:property name="y_offset" value="${-camera_width}" />
-        </xacro:if>
-        <link name="${bot_name}_camera_${position_name}_link">
+        <link name="${bot_name}_camera_link">
             <visual>
                 <geometry>
@@ -27,17 +20,17 @@
                             o_xyz="0 0 0" o_rpy="0 0 0" />
         </link>
-        <joint name="${bot_name}_${position_name}_base_camera_joint" type="fixed">
+        <joint name="${bot_name}_base_camera_joint" type="fixed">
             <parent link="${bot_name}_servo_link" />
-            <child link="${bot_name}_camera_${position_name}_link" />
+            <child link="${bot_name}_camera_link" />
             <origin xyz="-0.016 ${y_offset} 0.082" rpy="0 0.349 0" />
         </joint>
-        <link name="${bot_name}_camera_${position_name}_link_optical" />
-        <joint name="${bot_name}_${position_name}_optical_joint" type="fixed">
+        <link name="${bot_name}_camera_link_optical" />
+        <joint name="${bot_name}_optical_joint" type="fixed">
             <origin xyz="0 0 0" rpy="0 0 0"/>
-            <parent link="${bot_name}_camera_${position_name}_link"/>
-            <child link="${bot_name}_camera_${position_name}_link_optical"/>
+            <parent link="${bot_name}_camera_link"/>
+            <child link="${bot_name}_camera_link_optical"/>
         </joint>
-        <gazebo reference="${bot_name}_camera_${position_name}_link">
-            <sensor name="${bot_name}_camera_${position_name}" type="camera">
+        <gazebo reference="${bot_name}_camera_link">
+            <sensor name="${bot_name}_camera" type="camera">
                 <camera>
                     <horizontal_fov>1.3962634</horizontal_fov>
@@ -56,11 +49,11 @@
                         <stddev>0.007</stddev>
                     </noise>
-                    <optical_frame_id>${bot_name}_camera_${position_name}_link_optical</optical_frame_id>
-                    <camera_info_topic>${bot_name}_camera_${position_name}/camera_info</camera_info_topic>
+                    <optical_frame_id>${bot_name}_camera_link_optical</optical_frame_id>
+                    <camera_info_topic>${bot_name}_camera/camera_info</camera_info_topic>
                 </camera>
                 <always_on>1</always_on>
                 <update_rate>3</update_rate>
                 <visualize>true</visualize>
-                <topic>${bot_name}_camera_${position_name}/image_raw</topic>
+                <topic>${bot_name}_camera/image_raw</topic>
                 <plugin
                     filename="gz-sim-camera-system"

File: src/my_robot_description/urdf/ir.xacro (robot description, xacro)
@@ -1,9 +1,16 @@
 <?xml version="1.0"?>
 <robot xmlns:xacro="http://www.ros.org/wiki/xacro">
-<xacro:macro name="ir_sensor" params="bot_name" >
+<xacro:macro name="ir_sensor" params="bot_name position_name">
     <xacro:property name="ir_length" value="0.01" />
     <xacro:property name="ir_width" value="0.045" />
     <xacro:property name="ir_height" value="0.03" />
-    <link name="${bot_name}_ir_link">
+    <xacro:property name="y_offset" value="0.0" />
+    <xacro:if value="${position_name == 'L'}">
+        <xacro:property name="y_offset" value="${camera_width}" />
+    </xacro:if>
+    <xacro:if value="${position_name == 'R'}">
+        <xacro:property name="y_offset" value="${-camera_width}" />
+    </xacro:if>
+    <link name="${bot_name}_ir_${position_name}_link">
         <visual>
             <geometry>
@@ -20,17 +27,17 @@
                            o_xyz="0 0 0" o_rpy="0 0 0" />
     </link>
-    <joint name="${bot_name}_base_ir_joint" type="fixed">
+    <joint name="${bot_name}_${position_name}_base_ir_joint" type="fixed">
         <parent link="${bot_name}_base_link" />
-        <child link="${bot_name}_ir_link" />
+        <child link="${bot_name}_ir_${position_name}_link" />
         <origin xyz="0.084 0 -0.0275" rpy="0 ${pi/2} 0" />
     </joint>
-    <link name="${bot_name}_ir_link_optical" />
-    <joint name="${bot_name}_ir_optical_joint" type="fixed">
+    <link name="${bot_name}_ir_${position_name}_link_optical" />
+    <joint name="${bot_name}_ir_${position_name}_optical_joint" type="fixed">
         <origin xyz="0 0 0" rpy="${-pi/2} 0 ${-pi/2}"/>
-        <parent link="${bot_name}_ir_link"/>
-        <child link="${bot_name}_ir_link_optical"/>
+        <parent link="${bot_name}_ir_${position_name}_link"/>
+        <child link="${bot_name}_ir_${position_name}_link_optical"/>
     </joint>
-    <gazebo reference="${bot_name}_ir_link">
-        <sensor name="${bot_name}_ir" type="camera">
+    <gazebo reference="${bot_name}_ir_${position_name}_link">
+        <sensor name="${bot_name}_ir_${position_name}" type="camera">
             <camera>
                 <horizontal_fov>1.3962634</horizontal_fov>
@@ -49,11 +56,11 @@
                     <stddev>0.007</stddev>
                 </noise>
-                <optical_frame_id>${bot_name}_ir_link_optical</optical_frame_id>
-                <camera_info_topic>${bot_name}_ir/camera_info</camera_info_topic>
+                <optical_frame_id>${bot_name}_ir_${position_name}_link_optical</optical_frame_id>
+                <camera_info_topic>${bot_name}_ir_${position_name}/camera_info</camera_info_topic>
             </camera>
             <always_on>1</always_on>
             <update_rate>3</update_rate>
             <visualize>true</visualize>
-            <topic>${bot_name}_ir/image_raw</topic>
+            <topic>${bot_name}_ir_${position_name}/image_raw</topic>
             <plugin
                 filename="gz-sim-camera-system"

Commit message: x

File: src/my_robot_description/urdf/camera.xacro (robot description, xacro)
@@ -23,5 +23,5 @@
             <parent link="${bot_name}_servo_link" />
             <child link="${bot_name}_camera_link" />
-            <origin xyz="-0.016 ${y_offset} 0.082" rpy="0 0.349 0" />
+            <origin xyz="-0.016 0 0.082" rpy="0 0.349 0" />
         </joint>
         <link name="${bot_name}_camera_link_optical" />
