Commit message: ir positioning

File: src/my_robot_description/urdf/ir.xacro (robot description, xacro)
@@ -1,11 +1,11 @@
 <?xml version="1.0"?>
 <robot xmlns:xacro="http://www.ros.org/wiki/xacro">
-    <xacro:property name="camera_length" value="0.01" />
-    <xacro:property name="camera_width" value="0.05" />
-    <xacro:property name="camera_height" value="0.05" />
-    <link name="camera_linkBM">
+    <xacro:property name="ir_length" value="0.01" />
+    <xacro:property name="ir_width" value="0.045" />
+    <xacro:property name="ir_height" value="0.03" />
+    <link name="ir_linkBM">
         <visual>
             <geometry>
-                <box size="${camera_length} ${camera_width} ${camera_height}" />
+                <box size="${ir_length} ${ir_width} ${ir_height}" />
             </geometry>
             <material name="grey" />
@@ -13,24 +13,24 @@
         <collision>
             <geometry>
-                <box size="${camera_length} ${camera_width} ${camera_height}" />
+                <box size="${ir_length} ${ir_width} ${ir_height}" />
             </geometry>
         </collision>
-        <xacro:box_inertia m="0.1" x="${camera_length}" y="${camera_width}" z="${camera_height}"
+        <xacro:box_inertia m="0.1" x="${ir_length}" y="${ir_width}" z="${ir_height}"
                            o_xyz="0 0 0" o_rpy="0 0 0" />
     </link>
-    <joint name="base_camera_jointBM" type="fixed">
+    <joint name="base_ir_jointBM" type="fixed">
         <parent link="base_link" />
-        <child link="camera_linkBM" />
-        <origin xyz="0 0 ${base_height / 2.0 - 0.31}" rpy="0 ${pi/2} 0" />
+        <child link="ir_linkBM" />
+        <origin xyz="0.095 0 -0.01" rpy="0 ${pi/2} 0" />
     </joint>
-    <link name="camera_link_opticalBM" />
-    <joint name="camera_optical_jointBM" type="fixed">
+    <link name="ir_link_opticalBM" />
+    <joint name="ir_optical_jointBM" type="fixed">
         <origin xyz="0 0 0" rpy="${-pi/2} 0 ${-pi/2}"/>
-        <parent link="camera_linkBM"/>
-        <child link="camera_link_opticalBM"/>
+        <parent link="ir_linkBM"/>
+        <child link="ir_link_opticalBM"/>
     </joint>
-    <gazebo reference="camera_linkBM">
-        <sensor name="bm_camera" type="camera">
-            <camera>
+    <gazebo reference="ir_linkBM">
+        <sensor name="bm_ir" type="ir">
+            <ir>
                 <horizontal_fov>1.3962634</horizontal_fov>
                 <image>
@@ -48,14 +48,14 @@
                     <stddev>0.007</stddev>
                 </noise>
-                <optical_frame_id>camera_link_opticalBM</optical_frame_id>
-                <camera_info_topic>bm_camera/camera_info</camera_info_topic>
-            </camera>
+                <optical_frame_id>ir_link_opticalBM</optical_frame_id>
+                <ir_info_topic>bm_ir/ir_info</ir_info_topic>
+            </ir>
             <always_on>1</always_on>
             <update_rate>3</update_rate>
             <visualize>true</visualize>
-            <topic>bm_camera/image_raw</topic>
+            <topic>bm_ir/image_raw</topic>
             <plugin
-                filename="gz-sim-camera-system"
-                name="bm_camera_plugin"/>
+                filename="gz-sim-ir-system"
+                name="bm_ir_plugin"/>
         </sensor>
     </gazebo>

Commit message: model adjustments

File: src/my_robot_description/urdf/ir.xacro (robot description, xacro)
@@ -22,5 +22,5 @@
         <parent link="base_link" />
         <child link="ir_linkBM" />
-        <origin xyz="0.095 0 -0.01" rpy="0 ${pi/2} 0" />
+        <origin xyz="0.084 0 -0.0275" rpy="0 ${pi/2} 0" />
     </joint>
     <link name="ir_link_opticalBM" />

File: src/my_robot_description/urdf/mobile_base.xacro (robot description, xacro)
@@ -41,9 +41,9 @@
                     o_xyz="0 0 0" o_rpy="0 0 0"/>
         </link>
-        <!-- Front box -->
+        <!-- servo -->
         <joint name="servo_joint" type="continuous">
             <parent link="base_link"/>
             <child link="servo_link"/>
-            <origin xyz="0.09 0 0.03" rpy="0 0 0"/>
+            <origin xyz="0.076 0 0.03" rpy="0 0 0"/>
             <axis xyz="0 0 1"/>
         </joint>
@@ -52,5 +52,5 @@
                 <origin xyz="0 0 0" rpy="0 0 0"/>
                 <geometry>
-                    <box size="0.035 0.01 0.015"/>
+                    <box size="0.032 0.01 0.015"/>
                 </geometry>
                 <material name="accent_orange">
@@ -61,5 +61,5 @@
                 <origin xyz="0 0 0" rpy="0 0 0"/>
                 <geometry>
-                    <box size="0.035 0.01 0.015"/>
+                    <box size="0.032 0.01 0.015"/>
                 </geometry>
             </collision>
@@ -98,5 +98,5 @@
             <parent link="base_link"/>
             <child link="rear_left_wheel_link"/>
-            <origin xyz="-0.04 ${-(base_width/2.0) - 0.016} 0" rpy="0 0 0"/>
+            <origin xyz="-0.04 ${-(base_width/2.0) - 0.016} -0.005" rpy="0 0 0"/>
             <axis xyz="0 1 0"/>
         </joint>
@@ -104,5 +104,5 @@
             <parent link="base_link"/>
             <child link="rear_right_wheel_link"/>
-            <origin xyz="-0.04 ${(base_width/2.0) + 0.016} 0" rpy="0 0 0"/>
+            <origin xyz="-0.04 ${(base_width/2.0) + 0.016} -0.005" rpy="0 0 0"/>
             <axis xyz="0 1 0"/>
         </joint>
@@ -110,5 +110,5 @@
             <parent link="base_link"/>
             <child link="front_left_wheel_link"/>
-            <origin xyz="0.04 ${-(base_width/2.0) - 0.016} 0" rpy="0 0 0"/>
+            <origin xyz="0.04 ${-(base_width/2.0) - 0.016} -0.005" rpy="0 0 0"/>
             <axis xyz="0 1 0"/>
         </joint>
@@ -116,5 +116,5 @@
             <parent link="base_link"/>
             <child link="front_right_wheel_link"/>
-            <origin xyz="0.04 ${(base_width/2.0) + 0.016} 0" rpy="0 0 0"/>
+            <origin xyz="0.04 ${(base_width/2.0) + 0.016} -0.005" rpy="0 0 0"/>
             <axis xyz="0 1 0"/>
         </joint>

Commit message: Update ir.xacro

File: src/my_robot_description/urdf/ir.xacro (robot description, xacro)
@@ -4,5 +4,5 @@
     <xacro:property name="ir_width" value="0.045" />
     <xacro:property name="ir_height" value="0.03" />
-    <link name="ir_linkBM">
+    <link name="ir_link">
         <visual>
             <geometry>
@@ -19,18 +19,18 @@
                            o_xyz="0 0 0" o_rpy="0 0 0" />
     </link>
-    <joint name="base_ir_jointBM" type="fixed">
+    <joint name="base_ir_joint" type="fixed">
         <parent link="base_link" />
-        <child link="ir_linkBM" />
+        <child link="ir_link" />
         <origin xyz="0.084 0 -0.0275" rpy="0 ${pi/2} 0" />
     </joint>
-    <link name="ir_link_opticalBM" />
-    <joint name="ir_optical_jointBM" type="fixed">
+    <link name="ir_link_optical" />
+    <joint name="ir_optical_joint" type="fixed">
         <origin xyz="0 0 0" rpy="${-pi/2} 0 ${-pi/2}"/>
-        <parent link="ir_linkBM"/>
-        <child link="ir_link_opticalBM"/>
+        <parent link="ir_link"/>
+        <child link="ir_link_optical"/>
     </joint>
-    <gazebo reference="ir_linkBM">
-        <sensor name="bm_ir" type="camera">
-            <ir>
+    <gazebo reference="ir_link">
+        <sensor name="ir" type="camera">
+            <camera>
                 <horizontal_fov>1.3962634</horizontal_fov>
                 <image>
@@ -48,14 +48,14 @@
                     <stddev>0.007</stddev>
                 </noise>
-                <optical_frame_id>ir_link_opticalBM</optical_frame_id>
-                <ir_info_topic>bm_ir/ir_info</ir_info_topic>
-            </ir>
+                <optical_frame_id>ir_link_optical</optical_frame_id>
+                <ir_info_topic>camera/camera_info</ir_info_topic>
+            </camera>
             <always_on>1</always_on>
             <update_rate>3</update_rate>
             <visualize>true</visualize>
-            <topic>bm_ir/image_raw</topic>
+            <topic>camera/image_raw</topic>
             <plugin
                 filename="gz-sim-ir-system"
-                name="bm_ir_plugin"/>
+                name="camera_plugin"/>
         </sensor>
     </gazebo>

Commit message: x

File: src/my_robot_description/urdf/ir.xacro (robot description, xacro)
@@ -7,8 +7,8 @@
     <xacro:property name="y_offset" value="0.0" />
     <xacro:if value="${position_name == 'L'}">
-        <xacro:property name="y_offset" value="${camera_width}" />
+        <xacro:property name="y_offset" value="${ir_width}" />
     </xacro:if>
     <xacro:if value="${position_name == 'R'}">
-        <xacro:property name="y_offset" value="${-camera_width}" />
+        <xacro:property name="y_offset" value="${-ir_width}" />
     </xacro:if>
     <link name="${bot_name}_ir_${position_name}_link">

Commit message: x

File: src/my_robot_description/urdf/ir.xacro (robot description, xacro)
@@ -3,12 +3,12 @@
 <xacro:macro name="ir_sensor" params="bot_name position_name">
     <xacro:property name="ir_length" value="0.01" />
-    <xacro:property name="ir_width" value="0.045" />
-    <xacro:property name="ir_height" value="0.03" />
-    <xacro:property name="y_offset" value="0.0" />
+    <xacro:property name="ir_width" value="0.004" />
+    <xacro:property name="ir_height" value="0.006" />
+    <xacro:property name="y_offset" value="0.008" />
     <xacro:if value="${position_name == 'L'}">
-        <xacro:property name="y_offset" value="${ir_width}" />
+        <xacro:property name="y_offset" value="${0.008}" />
     </xacro:if>
     <xacro:if value="${position_name == 'R'}">
-        <xacro:property name="y_offset" value="${-ir_width}" />
+        <xacro:property name="y_offset" value="${-0.008}" />
     </xacro:if>
     <link name="${bot_name}_ir_${position_name}_link">

Commit message: x

File: src/my_robot_description/urdf/ir.xacro (robot description, xacro)
@@ -5,5 +5,5 @@
     <xacro:property name="ir_width" value="0.004" />
     <xacro:property name="ir_height" value="0.006" />
-    <xacro:property name="y_offset" value="0.008" />
+    <xacro:property name="y_offset" value="0.0" />
     <xacro:if value="${position_name == 'L'}">
         <xacro:property name="y_offset" value="${0.008}" />
@@ -12,4 +12,5 @@
         <xacro:property name="y_offset" value="${-0.008}" />
     </xacro:if>
+    <!-- else, M would be 0.0 -->
     <link name="${bot_name}_ir_${position_name}_link">
         <visual>
@@ -30,5 +31,5 @@
         <parent link="${bot_name}_base_link" />
         <child link="${bot_name}_ir_${position_name}_link" />
-        <origin xyz="0.084 0 -0.0275" rpy="0 ${pi/2} 0" />
+        <origin xyz="0.195 ${y_offset}} -0.0275" rpy="0 ${pi/2} 0" />
     </joint>
     <link name="${bot_name}_ir_${position_name}_link_optical" />

Commit message: x

File: src/my_robot_description/urdf/ir.xacro (robot description, xacro)
@@ -7,8 +7,8 @@
     <xacro:property name="y_offset" value="0.0" />
     <xacro:if value="${position_name == 'L'}">
-        <xacro:property name="y_offset" value="${0.008}" />
+        <xacro:property name="y_offset" value="0.008" />
     </xacro:if>
     <xacro:if value="${position_name == 'R'}">
-        <xacro:property name="y_offset" value="${-0.008}" />
+        <xacro:property name="y_offset" value="-0.008" />
     </xacro:if>
     <!-- else, M would be 0.0 -->

Commit message: x

File: src/my_robot_description/urdf/ir.xacro (robot description, xacro)
@@ -31,5 +31,5 @@
         <parent link="${bot_name}_base_link" />
         <child link="${bot_name}_ir_${position_name}_link" />
-        <origin xyz="0.195 ${y_offset}} -0.0275" rpy="0 ${pi/2} 0" />
+        <origin xyz="0.195 ${y_offset} -0.0275" rpy="0 ${pi/2} 0" />
     </joint>
     <link name="${bot_name}_ir_${position_name}_link_optical" />

Commit message: x

File: src/my_robot_description/urdf/ir.xacro (robot description, xacro)
@@ -31,5 +31,5 @@
         <parent link="${bot_name}_base_link" />
         <child link="${bot_name}_ir_${position_name}_link" />
-        <origin xyz="0.195 ${y_offset} -0.0275" rpy="0 ${pi/2} 0" />
+        <origin xyz="0.0885 ${y_offset} -0.0275" rpy="0 ${pi/2} 0" />
     </joint>
     <link name="${bot_name}_ir_${position_name}_link_optical" />
