Commit message: Moved rear and front wheel joint positions down (0.1)

File: src/my_robot_description/urdf/mobile_base.xacro (robot description, xacro)
@@ -191,5 +191,5 @@
         <parent link="base_link"/>
         <child link="rear_left_wheel_link"/>
-        <origin xyz="${(-(base_length + 0.01) / 2.0) + 0.2} 0.32 -0.1" rpy="0 0 0"/>
+        <origin xyz="${(-(base_length + 0.01) / 2.0) + 0.2} 0.32 -0.2" rpy="0 0 0"/>
         <axis xyz="0 1 0"/>
     </joint>
@@ -197,5 +197,5 @@
         <parent link="base_link"/>
         <child link="rear_right_wheel_link"/>
-        <origin xyz="${(-(base_length + 0.01) / 2.0) + 0.2} -0.32 -0.1" rpy="0 0 0"/>
+        <origin xyz="${(-(base_length + 0.01) / 2.0) + 0.2} -0.32 -0.2" rpy="0 0 0"/>
         <axis xyz="0 1 0"/>
     </joint>
@@ -206,5 +206,5 @@
         <parent link="base_link"/>
         <child link="front_right_wheel_link"/>
-        <origin xyz="${((base_length + 0.01) / 2.0) - 0.2} -0.32 -0.1" rpy="0 0 0"/>
+        <origin xyz="${((base_length + 0.01) / 2.0) - 0.2} -0.32 -0.2" rpy="0 0 0"/>
         <axis xyz="0 1 0"/>
     </joint>
@@ -230,5 +230,5 @@
         <parent link="base_link"/>
         <child link="front_left_wheel_link"/>
-        <origin xyz="${((base_length + 0.01) / 2.0) - 0.2} 0.32 -0.1" rpy="0 0 0"/>
+        <origin xyz="${((base_length + 0.01) / 2.0) - 0.2} 0.32 -0.2" rpy="0 0 0"/>
         <axis xyz="0 1 0"/>
     </joint>

Commit message: made the robot smaller

File: src/my_robot_description/urdf/mobile_base.xacro (robot description, xacro)
@@ -2,5 +2,5 @@
 <robot xmlns:xacro="http://www.ros.org/wiki/xacro">
     <!-- Updated properties to match your robot model -->
-    <xacro:property name="base_length" value="0.8"/>
+    <xacro:property name="base_length" value="0.6"/>
     <xacro:property name="base_width"  value="0.6"/>
     <xacro:property name="base_height" value="0.3"/>

Commit message: Made robot length from 0.8 to 0.7 and fixed wheels size

File: src/my_robot_description/urdf/mobile_base.xacro (robot description, xacro)
@@ -2,8 +2,8 @@
 <robot xmlns:xacro="http://www.ros.org/wiki/xacro">
     <!-- Updated properties to match your robot model -->
-    <xacro:property name="base_length" value="0.6"/>
-    <xacro:property name="base_width"  value="0.6"/>
+    <xacro:property name="base_length" value="0.7"/>
+    <xacro:property name="base_width"  value="0.5"/>
     <xacro:property name="base_height" value="0.3"/>
-    <xacro:property name="wheel_radius" value="0.15"/>
+    <xacro:property name="wheel_radius" value="0.125"/>
     <xacro:property name="wheel_length" value="0.1"/>
     <!-- ========================= -->
@@ -68,5 +68,5 @@
         <parent link="base_link"/>
         <child link="basket_back_link"/>
-        <origin xyz="-0.35 0 0.2" rpy="0 0 0"/>
+        <origin xyz="-0.3 0 0.2" rpy="0 0 0"/>
     </joint>
     <link name="basket_back_link">
@@ -84,5 +84,5 @@
         <parent link="base_link"/>
         <child link="basket_left_link"/>
-        <origin xyz="-0.2 0.2 0.2" rpy="0 0 0"/>
+        <origin xyz="-0.15 0.2 0.2" rpy="0 0 0"/>
     </joint>
     <link name="basket_left_link">
@@ -100,5 +100,5 @@
         <parent link="base_link"/>
         <child link="basket_right_link"/>
-        <origin xyz="-0.2 -0.2 0.2" rpy="0 0 0"/>
+        <origin xyz="-0.15 -0.2 0.2" rpy="0 0 0"/>
     </joint>
     <link name="basket_right_link">
@@ -116,5 +116,5 @@
         <parent link="base_link"/>
         <child link="basket_front_link"/>
-        <origin xyz="-0.05 0 0.2" rpy="0 0 0"/>
+        <origin xyz="0 0 0.2" rpy="0 0 0"/>
     </joint>
     <link name="basket_front_link">
@@ -191,5 +191,5 @@
         <parent link="base_link"/>
         <child link="rear_left_wheel_link"/>
-        <origin xyz="${(-(base_length + 0.01) / 2.0) + 0.2} 0.32 -0.15" rpy="0 0 0"/>
+        <origin xyz="${(-(base_length + 0.01) / 2.0) + 0.2} ${base_width/2.0} -0.15" rpy="0 0 0"/>
         <axis xyz="0 1 0"/>
     </joint>
@@ -197,5 +197,5 @@
         <parent link="base_link"/>
         <child link="rear_right_wheel_link"/>
-        <origin xyz="${(-(base_length + 0.01) / 2.0) + 0.2} -0.32 -0.15" rpy="0 0 0"/>
+        <origin xyz="${(-(base_length + 0.01) / 2.0) + 0.2} -${base_width/2.0} -0.15" rpy="0 0 0"/>
         <axis xyz="0 1 0"/>
     </joint>
@@ -206,5 +206,5 @@
         <parent link="base_link"/>
         <child link="front_right_wheel_link"/>
-        <origin xyz="${((base_length + 0.01) / 2.0) - 0.2} -0.32 -0.15" rpy="0 0 0"/>
+        <origin xyz="${((base_length + 0.01) / 2.0) - 0.2} -${base_width/2.0} -0.15" rpy="0 0 0"/>
         <axis xyz="0 1 0"/>
     </joint>
@@ -230,5 +230,5 @@
         <parent link="base_link"/>
         <child link="front_left_wheel_link"/>
-        <origin xyz="${((base_length + 0.01) / 2.0) - 0.2} 0.32 -0.15" rpy="0 0 0"/>
+        <origin xyz="${((base_length + 0.01) / 2.0) - 0.2} ${base_width/2.0} -0.15" rpy="0 0 0"/>
         <axis xyz="0 1 0"/>
     </joint>

Commit message: Made wheels bigger again (radius = 0.15)

File: src/my_robot_description/urdf/mobile_base.xacro (robot description, xacro)
@@ -5,5 +5,5 @@
     <xacro:property name="base_width"  value="0.5"/>
     <xacro:property name="base_height" value="0.3"/>
-    <xacro:property name="wheel_radius" value="0.125"/>
+    <xacro:property name="wheel_radius" value="0.15"/>
     <xacro:property name="wheel_length" value="0.1"/>
     <!-- ========================= -->

Commit message: made front wheels "fixed" and made the robot spawn a bit higher

File: src/my_robot_description/urdf/mobile_base.xacro (robot description, xacro)
@@ -203,5 +203,5 @@
     <!-- Front Wheels (Fixed)        -->
     <!-- ============================ -->
-    <joint name="front_right_wheel_joint" type="continuous">
+    <joint name="front_right_wheel_joint" type="fixed">
         <parent link="base_link"/>
         <child link="front_right_wheel_link"/>
@@ -227,5 +227,5 @@
                                 o_xyz="0 0 0" o_rpy="${pi/2.0} 0 0"/>
     </link>
-    <joint name="front_left_wheel_joint" type="continuous">
+    <joint name="front_left_wheel_joint" type="fixed">
         <parent link="base_link"/>
         <child link="front_left_wheel_link"/>

Commit message: changed front wheels back to continuous
- it doesn't actually help a lot but maybe it's better to have them be free rolling wheels.

File: src/my_robot_description/urdf/mobile_base.xacro (robot description, xacro)
@@ -203,5 +203,5 @@
     <!-- Front Wheels (Fixed)        -->
     <!-- ============================ -->
-    <joint name="front_right_wheel_joint" type="fixed">
+    <joint name="front_right_wheel_joint" type="continuous">
         <parent link="base_link"/>
         <child link="front_right_wheel_link"/>
@@ -227,5 +227,5 @@
                                 o_xyz="0 0 0" o_rpy="${pi/2.0} 0 0"/>
     </link>
-    <joint name="front_left_wheel_joint" type="fixed">
+    <joint name="front_left_wheel_joint" type="continuous">
         <parent link="base_link"/>
         <child link="front_left_wheel_link"/>

File: src/my_robot_description/urdf/mobile_base_gazebo.xacro (robot description, xacro)
@@ -26,5 +26,5 @@
             <left_joint>rear_left_wheel_joint</left_joint>
             <right_joint>rear_right_wheel_joint</right_joint>
-            <wheel_separation>0.44</wheel_separation>
+            <wheel_separation>0.4</wheel_separation>
             <wheel_radius>0.15</wheel_radius>
             <frame_id>odom</frame_id>

Commit message: Changing Robot wheels
not tested yet

File: src/my_robot_description/urdf/mobile_base.xacro (robot description, xacro)
@@ -188,4 +188,5 @@
     <xacro:rear_wheel_link prefix="rear_left"/>
     <xacro:rear_wheel_link prefix="rear_right"/>
+    <!--
     <joint name="rear_left_wheel_joint" type="continuous">
         <parent link="base_link"/>
@@ -200,7 +201,63 @@
         <axis xyz="0 1 0"/>
     </joint>
+    -->
+    <joint name="rear_left_wheel_joint" type="continuous">
+        <parent link="base_link"/>
+        <child link="rear_left_wheel_link"/>
+        <origin xyz="0 ${(base_width/2.0) - 0.03} -0.05" rpy="0 0 0"/>
+        <axis xyz="0 1 0"/>
+    </joint>
+    <joint name="rear_right_wheel_joint" type="continuous">
+        <parent link="base_link"/>
+        <child link="rear_right_wheel_link"/>
+        <origin xyz="0 ${-(base_width/2.0) + 0.03} -0.05" rpy="0 0 0"/>
+        <axis xyz="0 1 0"/>
+    </joint>
     <!-- ============================ -->
     <!-- Front Wheels (Fixed)        -->
     <!-- ============================ -->
+    <!--
+    <link name="front_right_wheel_link">
+        <visual>
+            <origin rpy="${pi/2} 0 0" xyz="0 0 0"/>
+            <geometry>
+                <cylinder length="${wheel_length}" radius="${wheel_radius}"/>
+            </geometry>
+            <material name="rubber_black">
+                <color rgba="0.06 0.06 0.06 1.0"/>
+            </material>
+        </visual>
+        <collision>
+            <geometry>
+                <sphere radius="${wheel_radius}"/>
+            </geometry>
+        </collision>
+        <xacro:cylinder_inertia m="1.0" r="${wheel_radius}" l="${wheel_length}"
+                                o_xyz="0 0 0" o_rpy="${pi/2.0} 0 0"/>
+    </link>
+    <link name="front_left_wheel_link">
+        <visual>
+            <origin rpy="${pi/2} 0 0" xyz="0 0 0"/>
+            <geometry>
+                <cylinder length="${wheel_length}" radius="${wheel_radius}"/>
+            </geometry>
+            <material name="rubber_black">
+                <color rgba="0.06 0.06 0.06 1.0"/>
+            </material>
+        </visual>
+        <collision>
+            <geometry>
+                <sphere radius="${wheel_radius}"/>
+            </geometry>
+        </collision>
+        <xacro:cylinder_inertia m="1.0" r="${wheel_radius}" l="${wheel_length}"
+                                o_xyz="0 0 0" o_rpy="${pi/2.0} 0 0"/>
+    </link>
+    <joint name="front_left_wheel_joint" type="continuous">
+        <parent link="base_link"/>
+        <child link="front_left_wheel_link"/>
+        <origin xyz="${((base_length + 0.01) / 2.0) - 0.15} ${(base_width/2.0) - 0.03} -0.05" rpy="0 0 0"/>
+        <axis xyz="0 1 0"/>
+    </joint>
     <joint name="front_right_wheel_joint" type="continuous">
         <parent link="base_link"/>
@@ -209,45 +266,32 @@
         <axis xyz="0 1 0"/>
     </joint>
-    <link name="front_right_wheel_link">
-        <visual>
-            <origin rpy="${pi/2} 0 0" xyz="0 0 0"/>
-            <geometry>
-                <cylinder length="${wheel_length}" radius="${wheel_radius}"/>
-            </geometry>
-            <material name="rubber_black">
-                <color rgba="0.06 0.06 0.06 1.0"/>
-            </material>
-        </visual>
-        <collision>
-            <geometry>
-                <sphere radius="${wheel_radius}"/>
-            </geometry>
-        </collision>
-        <xacro:cylinder_inertia m="1.0" r="${wheel_radius}" l="${wheel_length}"
-                                o_xyz="0 0 0" o_rpy="${pi/2.0} 0 0"/>
-    </link>
-    <joint name="front_left_wheel_joint" type="continuous">
-        <parent link="base_link"/>
-        <child link="front_left_wheel_link"/>
-        <origin xyz="${((base_length + 0.01) / 2.0) - 0.15} ${(base_width/2.0) - 0.03} -0.05" rpy="0 0 0"/>
-        <axis xyz="0 1 0"/>
-    </joint>
-    <link name="front_left_wheel_link">
-        <visual>
-            <origin rpy="${pi/2} 0 0" xyz="0 0 0"/>
-            <geometry>
-                <cylinder length="${wheel_length}" radius="${wheel_radius}"/>
-            </geometry>
-            <material name="rubber_black">
-                <color rgba="0.06 0.06 0.06 1.0"/>
-            </material>
-        </visual>
-        <collision>
-            <geometry>
-                <sphere radius="${wheel_radius}"/>
-            </geometry>
-        </collision>
-        <xacro:cylinder_inertia m="1.0" r="${wheel_radius}" l="${wheel_length}"
-                                o_xyz="0 0 0" o_rpy="${pi/2.0} 0 0"/>
+    -->
+    <joint name="front_caster_joint" type="fixed">
+        <parent link="base_link"/>
+        <child link="front_caster_link"/>
+        <origin xyz="0.3 0 -0.05" rpy="0 0 0"/>
+    </joint>
+    <link name="front_caster_link">
+        <visual>
+            <geometry><sphere radius="${wheel_radius}"/></geometry>
+            <material name="rubber_black"><color rgba="0.1 0.1 0.1 1"/></material>
+        </visual>
+        <collision>
+            <geometry><sphere radius="${wheel_radius}"/></collision>
+        <xacro:sphere_inertia m="0.5" r="${wheel_radius}" o_xyz="0 0 0" o_rpy="0 0 0"/>
+    </link>
+    <joint name="rear_caster_joint" type="fixed">
+        <parent link="base_link"/>
+        <child link="rear_caster_link"/>
+        <origin xyz="-0.3 0 -0.05" rpy="0 0 0"/>
+    </joint>
+    <link name="rear_caster_link">
+        <visual>
+            <geometry><sphere radius="${wheel_radius}"/></geometry>
+            <material name="rubber_black"><color rgba="0.1 0.1 0.1 1"/></material>
+        </visual>
+        <collision>
+            <geometry><sphere radius="${wheel_radius}"/></collision>
+        <xacro:sphere_inertia m="0.5" r="${wheel_radius}" o_xyz="0 0 0" o_rpy="0 0 0"/>
     </link>
 </robot>

File: src/my_robot_description/urdf/mobile_base_gazebo.xacro (robot description, xacro)
@@ -11,4 +11,5 @@
     </gazebo>
     <!--slippery front wheels-->
+    <!--
     <gazebo reference="front_left_wheel_link">
         <mu1 value="0.000" />
@@ -18,4 +19,11 @@
         <mu1 value="0.000" />
         <mu2 value="0.000" />
+    </gazebo>
+    -->
+    <gazebo reference="front_caster_link">
+        <mu1 value="0.0"/><mu2 value="0.0"/>
+    </gazebo>
+    <gazebo reference="rear_caster_link">
+        <mu1 value="0.0"/><mu2 value="0.0"/>
     </gazebo>
     <!-- Differential Drive Plugin -->

Commit message: caster wheels continuous and frictoinless

File: src/my_robot_description/urdf/mobile_base.xacro (robot description, xacro)
@@ -203,5 +203,5 @@
     <!-- Caster Wheels                -->
     <!-- ============================ -->
-    <joint name="front_caster_joint" type="fixed">
+    <joint name="front_caster_joint" type="continuous">
         <parent link="base_link"/>
         <child link="front_caster_link"/>
@@ -220,5 +220,5 @@
         <xacro:sphere_inertia m="0.5" r="${wheel_radius/1.5}" o_xyz="0 0 0" o_rpy="0 0 0"/>
     </link>
-    <joint name="rear_caster_joint" type="fixed">
+    <joint name="rear_caster_joint" type="continuous">
         <parent link="base_link"/>
         <child link="rear_caster_link"/>

File: src/my_robot_description/urdf/mobile_base_gazebo.xacro (robot description, xacro)
@@ -12,10 +12,10 @@
     <!--slippery front wheels-->
     <gazebo reference="front_caster_link">
-        <mu1 value="0.1"/>
-        <mu2 value="0.1"/>
+        <mu1 value="0"/>
+        <mu2 value="0"/>
     </gazebo>
     <gazebo reference="rear_caster_link">
-        <mu1 value="0.1"/>
-        <mu2 value="0.1"/>
+        <mu1 value="0"/>
+        <mu2 value="0"/>
     </gazebo>
     <!-- Differential Drive Plugin -->

Commit message: updating measurements of robot

File: src/my_robot_description/urdf/mobile_base.xacro (robot description, xacro)
@@ -2,9 +2,9 @@
 <robot xmlns:xacro="http://www.ros.org/wiki/xacro">
     <!-- Updated properties to match your robot model -->
-    <xacro:property name="base_length" value="0.7"/>
-    <xacro:property name="base_width"  value="0.5"/>
-    <xacro:property name="base_height" value="0.3"/>
-    <xacro:property name="wheel_radius" value="0.15"/>
-    <xacro:property name="wheel_length" value="0.1"/>
+    <xacro:property name="base_length" value="0.21"/>
+    <xacro:property name="base_width"  value="0.095"/>
+    <xacro:property name="base_height" value="0.045"/>
+    <xacro:property name="wheel_radius" value="0.032"/>
+    <xacro:property name="wheel_length" value="0.025"/>
     <!-- ========================= -->
     <!-- Base Footprint (empty)   -->
@@ -15,5 +15,5 @@
         <parent link="base_footprint"/>
         <child link="base_link"/>
-        <origin xyz="0 0 0.2"/>
+        <origin xyz="0 0 0.02"/>
     </joint>
     <!-- =============== -->
@@ -36,5 +36,5 @@
             <origin xyz="0 0 0"/>
         </collision>
-        <xacro:box_inertia m="5.0" x="${base_length}" y="${base_width}" z="${base_height}"
+        <xacro:box_inertia m="1.140" x="${base_length}" y="${base_width}" z="${base_height}"
                    o_xyz="0 0 0" o_rpy="0 0 0"/>
     </link>
@@ -43,5 +43,5 @@
         <parent link="base_link"/>
         <child link="front_box_link"/>
-        <origin xyz="0.18 0 0.20" rpy="0 0 0"/>
+        <origin xyz="0.125 0 0.20" rpy="0 0 0"/>
     </joint>
     <link name="front_box_link">
@@ -63,69 +63,4 @@
         <xacro:box_inertia m="1.0" x="0.4" y="0.4" z="0.3"
                    o_xyz="0 0 0" o_rpy="0 0 0"/>
-    </link>
-    <!-- Basket walls -->
-    <joint name="basket_back_joint" type="fixed">
-        <parent link="base_link"/>
-        <child link="basket_back_link"/>
-        <origin xyz="-0.3 0 0.2" rpy="0 0 0"/>
-    </joint>
-    <link name="basket_back_link">
-        <visual>
-            <origin xyz="0 0 0" rpy="0 0 0"/>
-            <geometry>
-                <box size="0.02 0.42 0.2"/>
-            </geometry>
-            <material name="wood_brown">
-                <color rgba="0.76 0.60 0.42 1.0"/>
-            </material>
-        </visual>
-    </link>
-    <joint name="basket_left_joint" type="fixed">
-        <parent link="base_link"/>
-        <child link="basket_left_link"/>
-        <origin xyz="-0.15 0.2 0.2" rpy="0 0 0"/>
-    </joint>
-    <link name="basket_left_link">
-        <visual>
-            <origin xyz="0 0 0" rpy="0 0 0"/>
-            <geometry>
-                <box size="0.3 0.02 0.2"/>
-            </geometry>
-            <material name="wood_brown">
-                <color rgba="0.76 0.60 0.42 1.0"/>
-            </material>
-        </visual>
-    </link>
-    <joint name="basket_right_joint" type="fixed">
-        <parent link="base_link"/>
-        <child link="basket_right_link"/>
-        <origin xyz="-0.15 -0.2 0.2" rpy="0 0 0"/>
-    </joint>
-    <link name="basket_right_link">
-        <visual>
-            <origin xyz="0 0 0" rpy="0 0 0"/>
-            <geometry>
-                <box size="0.3 0.02 0.2"/>
-            </geometry>
-            <material name="wood_brown">
-                <color rgba="0.76 0.60 0.42 1.0"/>
-            </material>
-        </visual>
-    </link>
-    <joint name="basket_front_joint" type="fixed">
-        <parent link="base_link"/>
-        <child link="basket_front_link"/>
-        <origin xyz="0 0 0.2" rpy="0 0 0"/>
-    </joint>
-    <link name="basket_front_link">
-        <visual>
-            <origin xyz="0 0 0" rpy="0 0 0"/>
-            <geometry>
-                <box size="0.02 0.42 0.2"/>
-            </geometry>
-            <material name="light_brown">
-                <color rgba="0.89 0.722 0.51 1"/>
-            </material>
-        </visual>
     </link>
     <!-- Headlights -->

Commit message: servo

File: src/my_robot_description/urdf/mobile_base.xacro (robot description, xacro)
@@ -40,14 +40,15 @@
     </link>
     <!-- Front box -->
-    <joint name="front_box_joint" type="fixed">
+    <joint name="servo_joint" type="continuous">
         <parent link="base_link"/>
-        <child link="front_box_link"/>
+        <child link="servo_link"/>
         <origin xyz="0.125 0 0.20" rpy="0 0 0"/>
+        <axis xyz="0 0 1"/>
     </joint>
-    <link name="front_box_link">
+    <link name="servo_link">
         <visual>
             <origin xyz="0 0 0" rpy="0 0 0"/>
             <geometry>
-                <box size="0.3 0.3 0.25"/>
+                <box size="0.035 0.01 0.015"/>
             </geometry>
             <material name="accent_orange">

Commit message: servo done

File: src/my_robot_description/urdf/mobile_base.xacro (robot description, xacro)
@@ -59,8 +59,8 @@
             <origin xyz="0 0 0" rpy="0 0 0"/>
             <geometry>
-                <box size="0.4 0.4 0.3"/>
+                <box size="0.035 0.01 0.015"/>
             </geometry>
         </collision>
-        <xacro:box_inertia m="1.0" x="0.4" y="0.4" z="0.3"
+        <xacro:box_inertia m="1.0" x="0.035" y="0.01" z="0.015"
                    o_xyz="0 0 0" o_rpy="0 0 0"/>
     </link>
