Commit message: finished mobile base urdf

File: src/my_robot_description/urdf/mobile_base.xacro (robot description, xacro)
@@ -1,173 +1,123 @@
 <?xml version="1.0"?>
-<robot xmlns:xacro="http://www.ros.org/wiki/xacro">
-    <!-- Updated properties to match your robot model -->
-    <xacro:property name="base_length" value="0.21"/>
-    <xacro:property name="base_width"  value="0.095"/>
-    <xacro:property name="base_height" value="0.045"/>
-    <xacro:property name="wheel_radius" value="0.032"/>
-    <xacro:property name="wheel_length" value="0.025"/>
-    <!-- ========================= -->
-    <!-- Base Footprint (empty)   -->
-    <!-- ========================= -->
-    <link name="base_footprint"/>
-    <!-- Fixed transform to base_link (body_link in your model) -->
-    <joint name="base_joint" type="fixed">
-        <parent link="base_footprint"/>
-        <child link="base_link"/>
-        <origin xyz="0 0 0.02"/>
-    </joint>
-    <!-- =============== -->
-    <!-- Base link body  -->
-    <!-- =============== -->
-    <link name="base_link">
-        <visual>
-            <geometry>
-                <box size="${base_length} ${base_width} ${base_height}"/>
-            </geometry>
-            <origin xyz="0 0 0"/>
-            <material name="body_blue">
-                <color rgba="0.09 0.46 0.71 1.0"/>
-            </material>
-        </visual>
-        <collision>
-            <geometry>
-                <box size="${base_length} ${base_width} ${base_height}"/>
-            </geometry>
-            <origin xyz="0 0 0"/>
-        </collision>
-        <xacro:box_inertia m="1.140" x="${base_length}" y="${base_width}" z="${base_height}"
-                   o_xyz="0 0 0" o_rpy="0 0 0"/>
-    </link>
-    <!-- Front box -->
-    <joint name="servo_joint" type="continuous">
-        <parent link="base_link"/>
-        <child link="servo_link"/>
-        <origin xyz="0.125 0 0.20" rpy="0 0 0"/>
-        <axis xyz="0 0 1"/>
-    </joint>
-    <link name="servo_link">
-        <visual>
-            <origin xyz="0 0 0" rpy="0 0 0"/>
-            <geometry>
-                <box size="0.035 0.01 0.015"/>
-            </geometry>
-            <material name="accent_orange">
-                <color rgba="0.95 0.47 0.14 1.0"/>
-            </material>
-        </visual>
-        <collision>
-            <origin xyz="0 0 0" rpy="0 0 0"/>
-            <geometry>
-                <box size="0.035 0.01 0.015"/>
-            </geometry>
-        </collision>
-        <xacro:box_inertia m="1.0" x="0.035" y="0.01" z="0.015"
-                   o_xyz="0 0 0" o_rpy="0 0 0"/>
-    </link>
-    <!-- Headlights -->
-    <joint name="light1_joint" type="fixed">
-        <parent link="base_link"/>
-        <child link="light1_link"/>
-        <origin xyz="${(base_length + 0.01) / 2.0} -0.15 0" rpy="0 -1.5708 0"/>
-    </joint>
-    <link name="light1_link">
-        <visual>
-            <origin xyz="0 0 0" rpy="0 0 0"/>
-            <geometry>
-                <cylinder length="0.01" radius="0.05"/>
-            </geometry>
-            <material name="headlight_warm">
-                <color rgba="1.00 0.96 0.84 1.0"/>
-            </material>
-        </visual>
-    </link>
-    <joint name="light2_joint" type="fixed">
-        <parent link="base_link"/>
-        <child link="light2_link"/>
-        <origin xyz="${(base_length + 0.01) / 2.0} 0.15 0" rpy="0 -1.5708 0"/>
-    </joint>
-    <link name="light2_link">
-        <visual>
-            <origin xyz="0 0 0" rpy="0 0 0"/>
-            <geometry>
-                <cylinder length="0.01" radius="0.05"/>
-            </geometry>
-            <material name="headlight_warm">
-                <color rgba="1.00 0.96 0.84 1.0"/>
-            </material>
-        </visual>
-    </link>
-    <!-- ============================ -->
-    <!-- Rear Wheels (Driven)        -->
-    <!-- ============================ -->
-    <xacro:macro name="rear_wheel_link" params="prefix">
-        <link name="${prefix}_wheel_link">
+<xacro:macro name="bot" params="bot_name">
+    <robot xmlns:xacro="http://www.ros.org/wiki/xacro">
+        <!-- Updated properties to match your robot model -->
+        <xacro:property name="base_length" value="0.21"/>
+        <xacro:property name="base_width"  value="0.095"/>
+        <xacro:property name="base_height" value="0.045"/>
+        <xacro:property name="wheel_radius" value="0.032"/>
+        <xacro:property name="wheel_length" value="0.025"/>
+        <!-- ========================= -->
+        <!-- Base Footprint (empty)   -->
+        <!-- ========================= -->
+        <link name="${bot_name}_base_footprint"/>
+        <!-- Fixed transform to base_link (body_link in your model) -->
+        <joint name="base_joint" type="fixed">
+            <parent link="base_footprint"/>
+            <child link="base_link"/>
+            <origin xyz="0 0 0.02"/>
+        </joint>
+        <!-- =============== -->
+        <!-- Base link body  -->
+        <!-- =============== -->
+        <link name="base_link">
             <visual>
                 <geometry>
-                    <cylinder radius="${wheel_radius}" length="${wheel_length}"/>
+                    <box size="${base_length} ${base_width} ${base_height}"/>
                 </geometry>
-                <origin xyz="0 0 0" rpy="${pi/2} 0 0"/>
-                <material name="rubber_black">
-                    <color rgba="0.06 0.06 0.06 1.0"/>
+                <origin xyz="0 0 0"/>
+                <material name="body_blue">
+                    <color rgba="0.09 0.46 0.71 1.0"/>
                 </material>
             </visual>
             <collision>
                 <geometry>
-                    <sphere radius="${wheel_radius}"/>
+                    <box size="${base_length} ${base_width} ${base_height}"/>
                 </geometry>
-                <origin xyz="0 0 0" rpy="${pi/2} 0 0"/>
+                <origin xyz="0 0 0"/>
             </collision>
-            <xacro:cylinder_inertia m="1.0" r="${wheel_radius}" l="${wheel_length}"
-                                    o_xyz="0 0 0" o_rpy="${pi/2.0} 0 0"/>
+            <xacro:box_inertia m="1.140" x="${base_length}" y="${base_width}" z="${base_height}"
+                    o_xyz="0 0 0" o_rpy="0 0 0"/>
         </link>
-    </xacro:macro>
-    <xacro:rear_wheel_link prefix="rear_left"/>
-    <xacro:rear_wheel_link prefix="rear_right"/>
-    <joint name="rear_left_wheel_joint" type="continuous">
-        <parent link="base_link"/>
-        <child link="rear_left_wheel_link"/>
-        <origin xyz="0 ${(base_width/2.0) + 0.03} -0.125" rpy="0 0 0"/>
-        <axis xyz="0 1 0"/>
-    </joint>
-    <joint name="rear_right_wheel_joint" type="continuous">
-        <parent link="base_link"/>
-        <child link="rear_right_wheel_link"/>
-        <origin xyz="0 ${-(base_width/2.0) - 0.03} -0.125" rpy="0 0 0"/>
-        <axis xyz="0 1 0"/>
-    </joint>
-    <!-- ============================ -->
-    <!-- Caster Wheels                -->
-    <!-- ============================ -->
-    <joint name="front_caster_joint" type="continuous">
-        <parent link="base_link"/>
-        <child link="front_caster_link"/>
-        <origin xyz="0.3 0 -0.175" rpy="0 0 0"/>
-    </joint>
-    <link name="front_caster_link">
-        <visual>
-            <geometry><sphere radius="${wheel_radius/1.5}"/></geometry>
-            <material name="rubber_black"><color rgba="0.1 0.1 0.1 1"/></material>
-        </visual>
-        <collision>
-            <geometry>
-            <sphere radius="${wheel_radius/1.5}"/>
-            </geometry>
-        </collision>
-        <xacro:sphere_inertia m="0.5" r="${wheel_radius/1.5}" o_xyz="0 0 0" o_rpy="0 0 0"/>
-    </link>
-    <joint name="rear_caster_joint" type="continuous">
-        <parent link="base_link"/>
-        <child link="rear_caster_link"/>
-        <origin xyz="-0.3 0 -0.175" rpy="0 0 0"/>
-    </joint>
-    <link name="rear_caster_link">
-        <visual>
-            <geometry><sphere radius="${wheel_radius/1.5}"/></geometry>
-            <material name="rubber_black"><color rgba="0.1 0.1 0.1 1"/></material>
-        </visual>
-        <collision>
-            <geometry><sphere radius="${wheel_radius/1.5}"/></geometry>
-        </collision>
-        <xacro:sphere_inertia m="0.5" r="${wheel_radius/1.5}" o_xyz="0 0 0" o_rpy="0 0 0"/>
-    </link>
-</robot>
+        <!-- Front box -->
+        <joint name="servo_joint" type="continuous">
+            <parent link="base_link"/>
+            <child link="servo_link"/>
+            <origin xyz="0.125 0 0.045" rpy="0 0 0"/>
+            <axis xyz="0 0 1"/>
+        </joint>
+        <link name="servo_link">
+            <visual>
+                <origin xyz="0 0 0" rpy="0 0 0"/>
+                <geometry>
+                    <box size="0.035 0.01 0.015"/>
+                </geometry>
+                <material name="accent_orange">
+                    <color rgba="0.95 0.47 0.14 1.0"/>
+                </material>
+            </visual>
+            <collision>
+                <origin xyz="0 0 0" rpy="0 0 0"/>
+                <geometry>
+                    <box size="0.035 0.01 0.015"/>
+                </geometry>
+            </collision>
+            <xacro:box_inertia m="1.0" x="0.035" y="0.01" z="0.015"
+                    o_xyz="0 0 0" o_rpy="0 0 0"/>
+        </link>
+        <!-- ============================ -->
+        <!-- Rear Wheels (Driven)        -->
+        <!-- ============================ -->
+        <xacro:macro name="wheel_link" params="prefix">
+            <link name="${prefix}_wheel_link">
+                <visual>
+                    <geometry>
+                        <cylinder radius="${wheel_radius}" length="${wheel_length}"/>
+                    </geometry>
+                    <origin xyz="0 0 0" rpy="${pi/2} 0 0"/>
+                    <material name="rubber_black">
+                        <color rgba="0.06 0.06 0.06 1.0"/>
+                    </material>
+                </visual>
+                <collision>
+                    <geometry>
+                        <sphere radius="${wheel_radius}"/>
+                    </geometry>
+                    <origin xyz="0 0 0" rpy="${pi/2} 0 0"/>
+                </collision>
+                <xacro:cylinder_inertia m="1.0" r="${wheel_radius}" l="${wheel_length}"
+                                        o_xyz="0 0 0" o_rpy="${pi/2.0} 0 0"/>
+            </link>
+        </xacro:macro>
+        <xacro:rear_wheel_link prefix="rear_left"/>
+        <xacro:rear_wheel_link prefix="rear_right"/>
+        <xacro:rear_wheel_link prefix="front_left"/>
+        <xacro:rear_wheel_link prefix="front_right"/>
+        <joint name="rear_left_wheel_joint" type="continuous">
+            <parent link="base_link"/>
+            <child link="rear_left_wheel_link"/>
+            <origin xyz="-0.04 ${-(base_width/2.0) - 0.016} -0.02" rpy="0 0 0"/>
+            <axis xyz="0 1 0"/>
+        </joint>
+        <joint name="rear_right_wheel_joint" type="continuous">
+            <parent link="base_link"/>
+            <child link="rear_right_wheel_link"/>
+            <origin xyz="-0.04 ${(base_width/2.0) + 0.016} -0.02" rpy="0 0 0"/>
+            <axis xyz="0 1 0"/>
+        </joint>
+        <joint name="front_left_wheel_joint" type="continuous">
+            <parent link="base_link"/>
+            <child link="rear_left_wheel_link"/>
+            <origin xyz="0.04 ${-(base_width/2.0) - 0.016} -0.02" rpy="0 0 0"/>
+            <axis xyz="0 1 0"/>
+        </joint>
+        <joint name="front_right_wheel_joint" type="continuous">
+            <parent link="base_link"/>
+            <child link="rear_right_wheel_link"/>
+            <origin xyz="0.04 ${(base_width/2.0) + 0.016} -0.02" rpy="0 0 0"/>
+            <axis xyz="0 1 0"/>
+        </joint>
+    </robot>
+</xacro:macro>
+<xacro:rear_wheel_link bot_name="twix"/>
+<xacro:rear_wheel_link bot_name="twirl"/>

Commit message: fixes

File: src/my_robot_description/urdf/mobile_base.xacro (robot description, xacro)
@@ -1,5 +1,5 @@
 <?xml version="1.0"?>
-<xacro:macro name="bot" params="bot_name">
-    <robot xmlns:xacro="http://www.ros.org/wiki/xacro">
+<!-- <xacro:macro name="bot" params="bot_name"> -->
+<robot xmlns:xacro="http://www.ros.org/wiki/xacro">
         <!-- Updated properties to match your robot model -->
         <xacro:property name="base_length" value="0.21"/>
@@ -11,5 +11,6 @@
         <!-- Base Footprint (empty)   -->
         <!-- ========================= -->
-        <link name="${bot_name}_base_footprint"/>
+        <!-- <link name="${bot_name}_base_footprint"/> -->
+        <link name="base_footprint"/>
         <!-- Fixed transform to base_link (body_link in your model) -->
         <joint name="base_joint" type="fixed">
@@ -90,8 +91,8 @@
             </link>
         </xacro:macro>
-        <xacro:rear_wheel_link prefix="rear_left"/>
-        <xacro:rear_wheel_link prefix="rear_right"/>
-        <xacro:rear_wheel_link prefix="front_left"/>
-        <xacro:rear_wheel_link prefix="front_right"/>
+        <xacro:wheel_link prefix="rear_left"/>
+        <xacro:wheel_link prefix="rear_right"/>
+        <xacro:wheel_link prefix="front_left"/>
+        <xacro:wheel_link prefix="front_right"/>
         <joint name="rear_left_wheel_joint" type="continuous">
             <parent link="base_link"/>
@@ -118,6 +119,6 @@
             <axis xyz="0 1 0"/>
         </joint>
-    </robot>
-</xacro:macro>
-<xacro:rear_wheel_link bot_name="twix"/>
-<xacro:rear_wheel_link bot_name="twirl"/>
+</robot>
+<!-- </xacro:macro> -->
+<!-- <xacro:rear_wheel_link bot_name="twix"/>
+<xacro:rear_wheel_link bot_name="twirl"/> -->

File: src/my_robot_description/urdf/mobile_base_gazebo.xacro (robot description, xacro)
@@ -10,10 +10,11 @@
         <mu2 value="1" />
     </gazebo>
-    <!--slippery front wheels-->
-    <gazebo reference="front_caster_link">
-        <mu1 value="0.0"/><mu2 value="0.0"/>
+     <gazebo reference="front_left_wheel_link">
+        <mu1 value="1" />
+        <mu2 value="1" />
     </gazebo>
-    <gazebo reference="rear_caster_link">
-        <mu1 value="0.0"/><mu2 value="0.0"/>
+    <gazebo reference="right_right_wheel_link">
+        <mu1 value="1" />
+        <mu2 value="1" />
     </gazebo>
     <!-- Differential Drive Plugin -->
@@ -24,6 +25,6 @@
             <left_joint>rear_left_wheel_joint</left_joint>
             <right_joint>rear_right_wheel_joint</right_joint>
-            <wheel_separation>0.56</wheel_separation>
-            <wheel_radius>0.15</wheel_radius>
+            <wheel_separation>0.124</wheel_separation>
+            <wheel_radius>0.032</wheel_radius>
             <max_wheel_torque>100</max_wheel_torque>
             <max_wheel_acceleration>2.0</max_wheel_acceleration>
@@ -39,6 +40,6 @@
             <joint_name>rear_left_wheel_joint</joint_name>
             <joint_name>rear_right_wheel_joint</joint_name>
-            <joint_name>rear_caster_joint</joint_name>
-            <joint_name>front_caster_joint</joint_name>
+            <joint_name>front_left_wheel_link</joint_name>
+            <joint_name>front_right_wheel_link</joint_name>
         </plugin>
     </gazebo>

Commit message: fixes

File: src/my_robot_description/urdf/mobile_base.xacro (robot description, xacro)
@@ -109,5 +109,5 @@
         <joint name="front_left_wheel_joint" type="continuous">
             <parent link="base_link"/>
-            <child link="rear_left_wheel_link"/>
+            <child link="front_left_wheel_link"/>
             <origin xyz="0.04 ${-(base_width/2.0) - 0.016} -0.02" rpy="0 0 0"/>
             <axis xyz="0 1 0"/>
@@ -115,5 +115,5 @@
         <joint name="front_right_wheel_joint" type="continuous">
             <parent link="base_link"/>
-            <child link="rear_right_wheel_link"/>
+            <child link="front_right_wheel_link"/>
             <origin xyz="0.04 ${(base_width/2.0) + 0.016} -0.02" rpy="0 0 0"/>
             <axis xyz="0 1 0"/>

Commit message: adjustments

File: src/my_robot_description/urdf/mobile_base.xacro (robot description, xacro)
@@ -45,5 +45,6 @@
             <parent link="base_link"/>
             <child link="servo_link"/>
-            <origin xyz="0.125 0 0.045" rpy="0 0 0"/>
+            <origin xyz="0.125 0 0.0225" rpy="0 0 0"/>
+            <!-- z was 0.045 -->
             <axis xyz="0 0 1"/>
         </joint>
@@ -98,5 +99,5 @@
             <parent link="base_link"/>
             <child link="rear_left_wheel_link"/>
-            <origin xyz="-0.04 ${-(base_width/2.0) - 0.016} -0.02" rpy="0 0 0"/>
+            <origin xyz="-0.04 ${-(base_width/2.0) - 0.016} 0" rpy="0 0 0"/>
             <axis xyz="0 1 0"/>
         </joint>
@@ -104,5 +105,5 @@
             <parent link="base_link"/>
             <child link="rear_right_wheel_link"/>
-            <origin xyz="-0.04 ${(base_width/2.0) + 0.016} -0.02" rpy="0 0 0"/>
+            <origin xyz="-0.04 ${(base_width/2.0) + 0.016} 0" rpy="0 0 0"/>
             <axis xyz="0 1 0"/>
         </joint>
@@ -110,5 +111,5 @@
             <parent link="base_link"/>
             <child link="front_left_wheel_link"/>
-            <origin xyz="0.04 ${-(base_width/2.0) - 0.016} -0.02" rpy="0 0 0"/>
+            <origin xyz="0.04 ${-(base_width/2.0) - 0.016} 0" rpy="0 0 0"/>
             <axis xyz="0 1 0"/>
         </joint>
@@ -116,5 +117,5 @@
             <parent link="base_link"/>
             <child link="front_right_wheel_link"/>
-            <origin xyz="0.04 ${(base_width/2.0) + 0.016} -0.02" rpy="0 0 0"/>
+            <origin xyz="0.04 ${(base_width/2.0) + 0.016} 0" rpy="0 0 0"/>
             <axis xyz="0 1 0"/>
         </joint>

Commit message: adjusted servo location

File: src/my_robot_description/urdf/mobile_base.xacro (robot description, xacro)
@@ -45,5 +45,5 @@
             <parent link="base_link"/>
             <child link="servo_link"/>
-            <origin xyz="0.125 0 0.0225" rpy="0 0 0"/>
+            <origin xyz="0.09 0 0.0225" rpy="0 0 0"/>
             <!-- z was 0.045 -->
             <axis xyz="0 0 1"/>

Commit message: x

File: src/my_robot_description/urdf/mobile_base.xacro (robot description, xacro)
@@ -64,5 +64,5 @@
         <!-- Rear Wheels (Driven)        -->
         <!-- ============================ -->
-        <xacro:macro name="${bot_name}_wheel_link" params="prefix">
+        <xacro:macro name="wheel_link" params="bot_name prefix">
             <link name="${bot_name}_${prefix}_wheel_link">
                 <visual>
@@ -83,8 +83,8 @@
             </link>
         </xacro:macro>
-        <xacro:wheel_link prefix="rear_left"/>
-        <xacro:wheel_link prefix="rear_right"/>
-        <xacro:wheel_link prefix="front_left"/>
-        <xacro:wheel_link prefix="front_right"/>
+        <xacro:wheel_link bot_name="${bot_name}" prefix="rear_left"/>
+        <xacro:wheel_link bot_name="${bot_name}" prefix="rear_right"/>
+        <xacro:wheel_link bot_name="${bot_name}" prefix="front_left"/>
+        <xacro:wheel_link bot_name="${bot_name}" prefix="front_right"/>
         <joint name="${bot_name}_rear_left_wheel_joint" type="continuous">
             <parent link="${bot_name}_base_link"/>

Commit message: separating wheels from base xacro file

File: src/my_robot_description/urdf/mobile_base.xacro (robot description, xacro)
@@ -1,5 +1,5 @@
 <?xml version="1.0"?>
 <robot xmlns:xacro="http://www.ros.org/wiki/xacro">
-<xacro:macro name="bot" params="bot_name" >
+    <xacro:macro name="bot" params="bot_name" >
         <!-- Updated properties to match your robot model -->
         <xacro:property name="base_length" value="0.21"/>
@@ -62,58 +62,9 @@
                     o_xyz="0 0 0" o_rpy="0 0 0"/>
         </link>
-        <!-- ============================ -->
-        <!-- Rear Wheels (Driven)        -->
-        <!-- ============================ -->
-        <xacro:macro name="wheel_link" params="bot_name prefix">
-            <link name="${bot_name}_${prefix}_wheel_link">
-                <visual>
-                    <geometry>
-                        <cylinder radius="${wheel_radius}" length="${wheel_length}"/>
-                    </geometry>
-                    <origin xyz="0 0 0" rpy="${pi/2} 0 0"/>
-                    <material name="rubber_black"/>
-                </visual>
-                <collision>
-                    <geometry>
-                        <sphere radius="${wheel_radius}"/>
-                    </geometry>
-                    <origin xyz="0 0 0" rpy="${pi/2} 0 0"/>
-                </collision>
-                <xacro:cylinder_inertia m="1.0" r="${wheel_radius}" l="${wheel_length}"
-                                        o_xyz="0 0 0" o_rpy="${pi/2.0} 0 0"/>
-            </link>
-        </xacro:macro>
-        <xacro:wheel_link bot_name="${bot_name}" prefix="rear_left"/>
-        <xacro:wheel_link bot_name="${bot_name}" prefix="rear_right"/>
-        <xacro:wheel_link bot_name="${bot_name}" prefix="front_left"/>
-        <xacro:wheel_link bot_name="${bot_name}" prefix="front_right"/>
-        <joint name="${bot_name}_rear_left_wheel_joint" type="continuous">
-            <parent link="${bot_name}_base_link"/>
-            <child link="${bot_name}_rear_left_wheel_link"/>
-            <origin xyz="-0.04 ${-(base_width/2.0) - 0.016} -0.005" rpy="0 0 0"/>
-            <axis xyz="0 1 0"/>
-        </joint>
-        <joint name="${bot_name}_rear_right_wheel_joint" type="continuous">
-            <parent link="${bot_name}_base_link"/>
-            <child link="${bot_name}_rear_right_wheel_link"/>
-            <origin xyz="-0.04 ${(base_width/2.0) + 0.016} -0.005" rpy="0 0 0"/>
-            <axis xyz="0 1 0"/>
-        </joint>
-        <joint name="${bot_name}_front_left_wheel_joint" type="continuous">
-            <parent link="${bot_name}_base_link"/>
-            <child link="${bot_name}_front_left_wheel_link"/>
-            <origin xyz="0.04 ${-(base_width/2.0) - 0.016} -0.005" rpy="0 0 0"/>
-            <axis xyz="0 1 0"/>
-        </joint>
-        <joint name="${bot_name}_front_right_wheel_joint" type="continuous">
-            <parent link="${bot_name}_base_link"/>
-            <child link="${bot_name}_front_right_wheel_link"/>
-            <origin xyz="0.04 ${(base_width/2.0) + 0.016} -0.005" rpy="0 0 0"/>
-            <axis xyz="0 1 0"/>
-        </joint>
-    <xacro:ir_sensor bot_name="${bot_name}"/>
-    <xacro:camera_sensor bot_name="${bot_name}"/>
-    <xacro:ultrasonic_sensor bot_name="${bot_name}"/>
-    <xacro:gazebo_file bot_name="${bot_name}"/>
-</xacro:macro>
+        <xacro:wheel bot_name="${bot_name}"/>
+        <xacro:ir_sensor bot_name="${bot_name}"/>
+        <xacro:camera_sensor bot_name="${bot_name}"/>
+        <xacro:ultrasonic_sensor bot_name="${bot_name}"/>
+        <xacro:gazebo_file bot_name="${bot_name}"/>
+    </xacro:macro>
 </robot>
