Commit message: x

File: src/my_robot_description/urdf/mobile_base.xacro (robot description, xacro)
@@ -62,5 +62,10 @@
                     o_xyz="0 0 0" o_rpy="0 0 0"/>
         </link>
+        <!-- wheels -->
         <xacro:wheel bot_name="${bot_name}"/>
+        <xacro:wheel_link bot_name="${bot_name}" prefix="rear_left" invert_x="-1" invert_y="-1"/>
+        <xacro:wheel_link bot_name="${bot_name}" prefix="rear_right" invert_x="-1" invert_y="1"/>
+        <xacro:wheel_link bot_name="${bot_name}" prefix="front_left" invert_x="1" invert_y="-1"/>
+        <xacro:wheel_link bot_name="${bot_name}" prefix="front_right" invert_x="1" invert_y="1"/>
         <xacro:ir_sensor bot_name="${bot_name}"/>
         <xacro:camera_sensor bot_name="${bot_name}"/>

File: src/my_robot_description/urdf/wheel.xacro (robot description, xacro)
@@ -1,5 +1,5 @@
 <?xml version="1.0"?>
 <robot xmlns:xacro="http://www.ros.org/wiki/xacro">
-    <xacro:macro name="wheel_link" params="bot_name prefix">
+    <xacro:macro name="wheel" params="bot_name prefix invert_x invert_y">
         <link name="${bot_name}_${prefix}_wheel_link">
             <visual>
@@ -19,34 +19,10 @@
                 o_xyz="0 0 0" o_rpy="${pi/2.0} 0 0"/>
         </link>
-    </xacro:macro>
-    <xacro:macro name="bot" params="bot_name" >
-        <xacro:wheel_link bot_name="${bot_name}" prefix="rear_left"/>
-        <xacro:wheel_link bot_name="${bot_name}" prefix="rear_right"/>
-        <xacro:wheel_link bot_name="${bot_name}" prefix="front_left"/>
-        <xacro:wheel_link bot_name="${bot_name}" prefix="front_right"/>
-    </xacro:macro>
-    <joint name="${bot_name}_rear_left_wheel_joint" type="continuous">
+        <joint name="${bot_name}_${prefix}_wheel_joint" type="continuous">
             <parent link="${bot_name}_base_link"/>
-            <child link="${bot_name}_rear_left_wheel_link"/>
-            <origin xyz="-0.04 ${-(base_width/2.0) - 0.016} -0.005" rpy="0 0 0"/>
+            <child link="${bot_name}_${prefix}_wheel_link"/>
+            <origin xyz="${invert_x*0.04} ${invert_y*(base_width/2.0) - 0.016} -0.005" rpy="0 0 0"/>
             <axis xyz="0 1 0"/>
         </joint>
-        <joint name="${bot_name}_rear_right_wheel_joint" type="continuous">
-            <parent link="${bot_name}_base_link"/>
-            <child link="${bot_name}_rear_right_wheel_link"/>
-            <origin xyz="-0.04 ${(base_width/2.0) + 0.016} -0.005" rpy="0 0 0"/>
-            <axis xyz="0 1 0"/>
-        </joint>
-        <joint name="${bot_name}_front_left_wheel_joint" type="continuous">
-            <parent link="${bot_name}_base_link"/>
-            <child link="${bot_name}_front_left_wheel_link"/>
-            <origin xyz="0.04 ${-(base_width/2.0) - 0.016} -0.005" rpy="0 0 0"/>
-            <axis xyz="0 1 0"/>
-        </joint>
-        <joint name="${bot_name}_front_right_wheel_joint" type="continuous">
-            <parent link="${bot_name}_base_link"/>
-            <child link="${bot_name}_front_right_wheel_link"/>
-            <origin xyz="0.04 ${(base_width/2.0) + 0.016} -0.005" rpy="0 0 0"/>
-            <axis xyz="0 1 0"/>
-        </joint>
+    </xacro:macro>
 </robot>

Commit message: x

File: src/my_robot_description/urdf/mobile_base.xacro (robot description, xacro)
@@ -17,4 +17,9 @@
             <child link="${bot_name}_base_link"/>
             <origin xyz="0 0 0.02"/>
+        </joint>
+        <joint name="${bot_name}_world_joint" type="floating">
+            <parent link="world"/>
+            <child link="${bot_name}_base_footprint"/>
+            <origin xyz="0 0 0"/>
         </joint>
         <!-- =============== -->

Commit message: fixing bridge

File: src/my_robot_description/urdf/mobile_base.xacro (robot description, xacro)
@@ -18,9 +18,9 @@
             <origin xyz="0 0 0.02"/>
         </joint>
-        <joint name="${bot_name}_world_joint" type="floating">
+        <!-- <joint name="${bot_name}_world_joint" type="floating">
             <parent link="world"/>
             <child link="${bot_name}_base_footprint"/>
             <origin xyz="0 0 0"/>
-        </joint>
+        </joint> -->
         <!-- =============== -->
         <!-- Base link body  -->

Commit message: x

File: src/my_robot_description/urdf/mobile_base.xacro (robot description, xacro)
@@ -18,9 +18,9 @@
             <origin xyz="0 0 0.02"/>
         </joint>
-        <!-- <joint name="${bot_name}_world_joint" type="floating">
+        <joint name="${bot_name}_world_joint" type="floating">
             <parent link="world"/>
             <child link="${bot_name}_base_footprint"/>
             <origin xyz="0 0 0"/>
-        </joint> -->
+        </joint>
         <!-- =============== -->
         <!-- Base link body  -->

Commit message: duplication finished

File: src/my_robot_description/urdf/mobile_base.xacro (robot description, xacro)
@@ -17,9 +17,4 @@
             <child link="${bot_name}_base_link"/>
             <origin xyz="0 0 0.02"/>
-        </joint>
-        <joint name="${bot_name}_world_joint" type="floating">
-            <parent link="world"/>
-            <child link="${bot_name}_base_footprint"/>
-            <origin xyz="0 0 0"/>
         </joint>
         <!-- =============== -->

Commit message: imu and lidar for sim

File: src/my_robot_description/urdf/mobile_base.xacro (robot description, xacro)
@@ -39,9 +39,16 @@
         </link>
         <!-- servo -->
-        <joint name="${bot_name}_servo_joint" type="continuous">
+        <!-- <joint name="${bot_name}_servo_joint" type="continuous">
             <parent link="${bot_name}_base_link"/>
             <child link="${bot_name}_servo_link"/>
             <origin xyz="0.076 0 0.03" rpy="0 0 0"/>
             <axis xyz="0 0 1"/>
+        </joint> -->
+        <joint name="${bot_name}_servo_joint" type="revolute">
+            <parent link="${bot_name}_base_link"/>
+            <child link="${bot_name}_servo_link"/>
+            <origin xyz="0.076 0 0.03" rpy="0 0 0"/>
+            <axis xyz="0 0 1"/>
+            <limit lower="-1.5708" upper="1.5708" effort="10.0" velocity="5.0"/>
         </joint>
         <link name="${bot_name}_servo_link">

Commit message: x

File: src/my_robot_description/urdf/mobile_base.xacro (robot description, xacro)
@@ -51,4 +51,5 @@
             <axis xyz="0 0 1"/>
             <limit lower="-1.5708" upper="1.5708" effort="10.0" velocity="5.0"/>
+            <dynamics damping="0.1" friction="0.05"/>
         </joint>
         <link name="${bot_name}_servo_link">

File: src/my_robot_description/urdf/mobile_base_gazebo.xacro (robot description, xacro)
@@ -50,13 +50,13 @@
         </gazebo>
         <!-- Servo Position Controller -->
-        <gazebo>
+        <gazebo reference="${bot_name}_base_link">
             <plugin
                 filename="gz-sim-joint-position-controller-system"
                 name="gz::sim::systems::JointPositionController">
                 <joint_name>${bot_name}_servo_joint</joint_name>
-                <topic>/${bot_name}/servo_cmd</topic>
-                <p_gain>20</p_gain>
+                <topic>${bot_name}/servo_cmd</topic>
+                <p_gain>10</p_gain>
                 <i_gain>0.0</i_gain>
-                <d_gain>0.5</d_gain>
+                <d_gain>0.1</d_gain>
                 <i_max>1</i_max>
                 <i_min>-1</i_min>
